File: citizen_sensor/citizen_sensor.sch (KiCad schematic (older format))
At the start: 20 parts

Commit message: charger
Parts:
- added C?: 47uf, symbol Device:C_Small
- added C?: 100nf, symbol Device:C_Small
- added C?: C_Small, symbol Device:C_Small
- added D?: CHARGE, symbol Device:LED
- added J?: BATT, symbol Connector:Screw_Terminal_01x02
- added R? (x3): R, symbol Device:R
- added U?: MCP73831, symbol electroniccats:MCP73831
Connections:
- wire segments 62 -> 93

Commit message: modulation LoRa
Parts:
- added C?: C_Small, symbol Device:C_Small
Connections:
- net labels added: DIO0, DIO1, DIO2, DIO5, MISO, MOSI, RFM_RST, SCK, SS
- wire segments 93 -> 104
- no-connect marks 0 -> 3
Other:
- note added: "Modulation LoRa\n"
Changed lines of the file:
@@
 L RF_AM_FM:RFM95W-868S2 U?
 U 1 1 5C48B732
-P 1840 4570
-F 0 "U?" H 1840 5248 50  0000 C CNN
-F 1 "RFM95W-868S2" H 1840 5157 50  0000 C CNN
-F 2 "" H -1460 6220 50  0001 C CNN
-F 3 "http://www.hoperf.com/upload/rf/RFM95_96_97_98W.pdf" H -1460 6220 50  0001 C CNN
-	1    1840 4570
+P 9080 5000
+F 0 "U?" H 8750 5460 50  0000 C CNN
+F 1 "RFM95W-868S2" H 8590 4400 50  0000 C CNN
+F 2 "" H 5780 6650 50  0001 C CNN
+F 3 "http://www.hoperf.com/upload/rf/RFM95_96_97_98W.pdf" H 5780 6650 50  0001 C CNN
+	1    9080 5000
 	1    0    0    -1
 $EndComp
@@
 L Sensor:BME280 U?
 U 1 1 5C48BD79
-P 5610 6460
-F 0 "U?" H 5180 6506 50  0000 R CNN
-F 1 "BME280" H 5180 6415 50  0000 R CNN
-F 2 "Package_LGA:Bosch_LGA-8_2.5x2.5mm_P0.65mm_ClockwisePinNumbering" H 5610 6260 50  0001 C CNN
-F 3 "https://ae-bst.resource.bosch.com/media/_tech/media/datasheets/BST-BME280_DS001-11.pdf" H 5610 6260 50  0001 C CNN
-	1    5610 6460
-	1    0    0    -1
+P 4510 4300
+F 0 "U?" V 4040 4620 50  0000 R CNN
+F 1 "BME280" V 4040 4180 50  0000 R CNN
+F 2 "Package_LGA:Bosch_LGA-8_2.5x2.5mm_P0.65mm_ClockwisePinNumbering" H 4510 4100 50  0001 C CNN
+F 3 "https://ae-bst.resource.bosch.com/media/_tech/media/datasheets/BST-BME280_DS001-11.pdf" H 4510 4100 50  0001 C CNN
+	1    4510 4300
+	0    1    1    0
 $EndComp
 $Comp
@@
 L Device:Antenna_Shield AE?
 U 1 1 5C48C2A7
-P 4080 4040
-F 0 "AE?" H 4220 4081 50  0000 L CNN
-F 1 "Antenna_Shield" H 4220 3990 50  0000 L CNN
-F 2 "" H 4080 4140 50  0001 C CNN
-F 3 "~" H 4080 4140 50  0001 C CNN
-	1    4080 4040
+P 9860 4380
+F 0 "AE?" H 10000 4421 50  0000 L CNN
+F 1 "Antenna_Shield" H 10000 4330 50  0000 L CNN
+F 2 "" H 9860 4480 50  0001 C CNN
+F 3 "~" H 9860 4480 50  0001 C CNN
+	1    9860 4380
 	1    0    0    -1
 $EndComp
@@
 L electroniccats:VEML6075 U?
 U 1 1 5C48D32D
-P 8669 5335
-F 0 "U?" H 8669 5576 50  0000 C CNN
-F 1 "VEML6075" H 8669 5075 50  0000 C CNN
-F 2 "" H 8669 5335 50  0001 C CNN
-F 3 "" H 8669 5335 50  0001 C CNN
-	1    8669 5335
+P 1560 4540
+F 0 "U?" H 1560 4781 50  0000 C CNN
+F 1 "VEML6075" H 1560 4280 50  0000 C CNN
+F 2 "" H 1560 4540 50  0001 C CNN
+F 3 "" H 1560 4540 50  0001 C CNN
+	1    1560 4540
 	1    0    0    -1
 $EndComp
@@
 L electroniccats:MICS-4514 U?
 U 1 1 5C48BCB3
-P 1780 7090
-F 0 "U?" H 1780 7557 50  0000 C CNN
-F 1 "MICS-4514" H 1780 7466 50  0000 C CNN
-F 2 "MICS_10-SMD" H 1730 6790 50  0001 L BNN
-F 3 "None" H 1730 6790 50  0001 L BNN
-F 4 "None" H 1730 6790 50  0001 L BNN "Field5"
-	1    1780 7090
+P 1690 6800
+F 0 "U?" H 1690 7267 50  0000 C CNN
+F 1 "MICS-4514" H 1690 7176 50  0000 C CNN
+F 2 "MICS_10-SMD" H 1640 6500 50  0001 L BNN
+F 3 "None" H 1640 6500 50  0001 L BNN
+F 4 "None" H 1640 6500 50  0001 L BNN "Field5"
+	1    1690 6800
 	1    0    0    -1
 $EndComp
@@
 L Connector:Conn_01x02_Female J?
 U 1 1 5C48C861
-P 3380 7050
-F 0 "J?" H 3407 7026 50  0000 L CNN
-F 1 "POM-3044P-R" H 3407 6935 50  0000 L CNN
-F 2 "" H 3380 7050 50  0001 C CNN
-F 3 "~" H 3380 7050 50  0001 C CNN
-	1    3380 7050
+P 3990 6680
+F 0 "J?" H 4017 6656 50  0000 L CNN
+F 1 "POM-3044P-R" H 4017 6565 50  0000 L CNN
+F 2 "" H 3990 6680 50  0001 C CNN
+F 3 "~" H 3990 6680 50  0001 C CNN
+	1    3990 6680
 	1    0    0    -1
 $EndComp
@@
 Wire Notes Line
 	470  3600 11200 3600
+$Comp
+L power:+3.3V #PWR?
+U 1 1 5C4E30EB
+P 9080 4400
+F 0 "#PWR?" H 9080 4250 50  0001 C CNN
+F 1 "+3.3V" H 9095 4573 50  0000 C CNN
+F 2 "" H 9080 4400 50  0001 C CNN
+F 3 "" H 9080 4400 50  0001 C CNN
+	1    9080 4400
+	1    0    0    -1
+$EndComp
+$Comp
+L power:GND #PWR?
+U 1 1 5C4E38A3
+P 9080 5700
+F 0 "#PWR?" H 9080 5450 50  0001 C CNN
+F 1 "GND" H 9085 5527 50  0000 C CNN
+F 2 "" H 9080 5700 50  0001 C CNN
+F 3 "" H 9080 5700 50  0001 C CNN
+	1    9080 5700
+	1    0    0    -1
+$EndComp
+Wire Wire Line
+	8980 5600 8980 5700
+Wire Wire Line
+	8980 5700 9080 5700
+Wire Wire Line
+	9180 5600 9180 5700
+Wire Wire Line
+	9180 5700 9080 5700
+Connection ~ 9080 5700
+Wire Wire Line
+	9080 5600 9080 5700
+Wire Wire Line
+	9580 4700 9860 4700
+Wire Wire Line
+	9860 4700 9860 4580
+Wire Wire Line
+	9080 4400 9080 4500
+$Comp
+L Device:C_Small C?
+U 1 1 5C4F27C7
+P 7780 4990
+F 0 "C?" H 7872 5036 50  0000 L CNN
+F 1 "C_Small" H 7872 4945 50  0000 L CNN
+F 2 "" H 7780 4990 50  0001 C CNN
+F 3 "~" H 7780 4990 50  0001 C CNN
+	1    7780 4990
+	1    0    0    -1
+$EndComp
+$Comp
+L power:GND #PWR?
+U 1 1 5C4F28F1
+P 7780 5210
+F 0 "#PWR?" H 7780 4960 50  0001 C CNN
+F 1 "GND" H 7785 5037 50  0000 C CNN
+F 2 "" H 7780 5210 50  0001 C CNN
+F 3 "" H 7780 5210 50  0001 C CNN
+	1    7780 5210
+	1    0    0    -1
+$EndComp
+$Comp
+L power:+3.3V #PWR?
+U 1 1 5C4F2997
+P 7780 4830
+F 0 "#PWR?" H 7780 4680 50  0001 C CNN
+F 1 "+3.3V" H 7795 5003 50  0000 C CNN
+F 2 "" H 7780 4830 50  0001 C CNN
+F 3 "" H 7780 4830 50  0001 C CNN
+	1    7780 4830
+	1    0    0    -1
+$EndComp
+Wire Wire Line
+	7780 4830 7780 4890
+Wire Wire Line
+	7780 5090 7780 5210
+$Comp
+L power:GND #PWR?
+U 1 1 5C4F90B3
+P 9960 4720
+F 0 "#PWR?" H 9960 4470 50  0001 C CNN
+F 1 "GND" H 9965 4547 50  0000 C CNN
+F 2 "" H 9960 4720 50  0001 C CNN
+F 3 "" H 9960 4720 50  0001 C CNN
+	1    9960 4720
+	1    0    0    -1
+$EndComp
+Wire Wire Line
+	9960 4580 9960 4720
+Wire Notes Line
+	6970 6530 6970 3600
+Text Label 8580 4700 2    50   ~ 0
+SCK
+Text Label 8580 4800 2    50   ~ 0
+MOSI
+Text Label 8580 4900 2    50   ~ 0
+MISO
+Text Label 8580 5000 2    50   ~ 0
+SS
+Text Label 8580 5200 2    50   ~ 0
+RFM_RST
+Text Label 9580 4900 0    50   ~ 0
+DIO5
+Text Label 9580 5200 0    50   ~ 0
+DIO2
+Text Label 9580 5300 0    50   ~ 0
+DIO1
+NoConn ~ 9580 5000
+NoConn ~ 9580 5100
+Text Label 9580 5400 0    50   ~ 0
+DIO0
+Text Notes 7000 3680 0    50   ~ 0
+Modulation LoRa\n
+Text Label 7300 2100 2    50   ~ 0
+DIO0
+Text Label 8700 2100 0    50   ~ 0
+DIO2
+Text Label 8700 2200 0    50   ~ 0
+D+
+Text Label 8700 2300 0    50   ~ 0
+D-
+Text Label 8700 2400 0    50   ~ 0
+DIO1
+Text Label 8700 2500 0    50   ~ 0
+MISO
+Text Label 8700 2800 0    50   ~ 0
+SS
+Text Label 8700 2600 0    50   ~ 0
+SCK
+Text Label 8700 2700 0    50   ~ 0
+MOSI
+Text Label 8700 2900 0    50   ~ 0
+RFM_RST
+Text Label 8700 3000 0    50   ~ 0
+DIO5
+NoConn ~ 8700 2000
 $EndSCHEMATC

Commit message: values capacitor and resistor
Parts:
- C?: value C_Small -> 10uf
- C?: value C_Small -> 0.1uf
- R? (x2): value R -> 10k
- R? (x2): value R -> 1k
Changed lines of the file:
@@
 U 1 1 5C48B93D
 P 5220 1105
-F 0 "D?" H 5211 1321 50  0000 C CNN
-F 1 "ON" H 5211 1230 50  0000 C CNN
+F 0 "D?" V 5235 1255 50  0000 C CNN
+F 1 "ON" V 5145 1255 50  0000 C CNN
 F 2 "" H 5220 1105 50  0001 C CNN
 F 3 "~" H 5220 1105 50  0001 C CNN
@@
 L Sensor:BME280 U?
 U 1 1 5C48BD79
-P 4510 4300
-F 0 "U?" V 4040 4620 50  0000 R CNN
-F 1 "BME280" V 4040 4180 50  0000 R CNN
-F 2 "Package_LGA:Bosch_LGA-8_2.5x2.5mm_P0.65mm_ClockwisePinNumbering" H 4510 4100 50  0001 C CNN
-F 3 "https://ae-bst.resource.bosch.com/media/_tech/media/datasheets/BST-BME280_DS001-11.pdf" H 4510 4100 50  0001 C CNN
-	1    4510 4300
+P 5220 4660
+F 0 "U?" V 4750 4980 50  0000 R CNN
+F 1 "BME280" V 4750 4540 50  0000 R CNN
+F 2 "Package_LGA:Bosch_LGA-8_2.5x2.5mm_P0.65mm_ClockwisePinNumbering" H 5220 4460 50  0001 C CNN
+F 3 "https://ae-bst.resource.bosch.com/media/_tech/media/datasheets/BST-BME280_DS001-11.pdf" H 5220 4460 50  0001 C CNN
+	1    5220 4660
 	0    1    1    0
 $EndComp
@@
 L Connector:Conn_01x02_Female J?
 U 1 1 5C48C861
-P 3990 6680
-F 0 "J?" H 4017 6656 50  0000 L CNN
-F 1 "POM-3044P-R" H 4017 6565 50  0000 L CNN
-F 2 "" H 3990 6680 50  0001 C CNN
-F 3 "~" H 3990 6680 50  0001 C CNN
-	1    3990 6680
+P 5030 6830
+F 0 "J?" H 5057 6806 50  0000 L CNN
+F 1 "POM-3044P-R" H 5057 6715 50  0000 L CNN
+F 2 "" H 5030 6830 50  0001 C CNN
+F 3 "~" H 5030 6830 50  0001 C CNN
+	1    5030 6830
 	1    0    0    -1
 $EndComp
@@
 P 5220 1480
 F 0 "R?" H 5290 1526 50  0000 L CNN
-F 1 "R" H 5290 1435 50  0000 L CNN
+F 1 "1k" H 5290 1435 50  0000 L CNN
 F 2 "" V 5150 1480 50  0001 C CNN
 F 3 "~" H 5220 1480 50  0001 C CNN
@@
 P 2690 2790
 F 0 "R?" V 2610 2790 50  0000 C CNN
-F 1 "R" V 2770 2790 50  0000 C CNN
+F 1 "10k" V 2770 2790 50  0000 C CNN
 F 2 "" V 2620 2790 50  0001 C CNN
 F 3 "~" H 2690 2790 50  0001 C CNN
@@
 U 1 1 5C495CD1
 P 3930 2890
-F 0 "R?" V 4000 2936 50  0000 L CNN
-F 1 "R" V 4000 2845 50  0000 L CNN
+F 0 "R?" V 4010 2860 50  0000 L CNN
+F 1 "10k" V 3840 2830 50  0000 L CNN
 F 2 "" V 3860 2890 50  0001 C CNN
 F 3 "~" H 3930 2890 50  0001 C CNN
@@
 P 4210 3040
 F 0 "C?" H 4302 3086 50  0000 L CNN
-F 1 "C_Small" H 4302 2995 50  0000 L CNN
+F 1 "10uf" H 4302 2995 50  0000 L CNN
 F 2 "" H 4210 3040 50  0001 C CNN
 F 3 "~" H 4210 3040 50  0001 C CNN
@@
 P 3720 2270
 F 0 "R?" V 3630 2270 50  0000 C CNN
-F 1 "R" V 3820 2270 50  0000 C CNN
+F 1 "1k" V 3820 2270 50  0000 C CNN
 F 2 "" V 3650 2270 50  0001 C CNN
 F 3 "~" H 3720 2270 50  0001 C CNN
@@
 P 7780 4990
 F 0 "C?" H 7872 5036 50  0000 L CNN
-F 1 "C_Small" H 7872 4945 50  0000 L CNN
+F 1 "0.1uf" H 7872 4945 50  0000 L CNN
 F 2 "" H 7780 4990 50  0001 C CNN
 F 3 "~" H 7780 4990 50  0001 C CNN

Commit message: light sensor
Parts:
- added C?: 0.1uf, symbol Device:C_Small
- added D?: Light ON, symbol Device:LED
- added R?: 1k, symbol Device:R
- added R? (x2): 2.2k, symbol Device:R
Connections:
- net labels added: SCL, SDA
- wire segments 104 -> 123
Other:
- note added: "7-bit Unshifted I2C Address 0x10"
- note added: "Light Sensor"
- note added: "Module LoRa\n"
- note removed: "Modulation LoRa\n"
Changed lines of the file:
@@
 L Sensor:BME280 U?
 U 1 1 5C48BD79
-P 5220 4660
-F 0 "U?" V 4750 4980 50  0000 R CNN
-F 1 "BME280" V 4750 4540 50  0000 R CNN
-F 2 "Package_LGA:Bosch_LGA-8_2.5x2.5mm_P0.65mm_ClockwisePinNumbering" H 5220 4460 50  0001 C CNN
-F 3 "https://ae-bst.resource.bosch.com/media/_tech/media/datasheets/BST-BME280_DS001-11.pdf" H 5220 4460 50  0001 C CNN
-	1    5220 4660
+P 5770 4510
+F 0 "U?" V 5300 4830 50  0000 R CNN
+F 1 "BME280" V 5300 4390 50  0000 R CNN
+F 2 "Package_LGA:Bosch_LGA-8_2.5x2.5mm_P0.65mm_ClockwisePinNumbering" H 5770 4310 50  0001 C CNN
+F 3 "https://ae-bst.resource.bosch.com/media/_tech/media/datasheets/BST-BME280_DS001-11.pdf" H 5770 4310 50  0001 C CNN
+	1    5770 4510
 	0    1    1    0
 $EndComp
@@
 L electroniccats:VEML6075 U?
 U 1 1 5C48D32D
-P 1560 4540
-F 0 "U?" H 1560 4781 50  0000 C CNN
-F 1 "VEML6075" H 1560 4280 50  0000 C CNN
-F 2 "" H 1560 4540 50  0001 C CNN
-F 3 "" H 1560 4540 50  0001 C CNN
-	1    1560 4540
+P 2210 4520
+F 0 "U?" H 2210 4761 50  0000 C CNN
+F 1 "VEML6075" H 2210 4260 50  0000 C CNN
+F 2 "" H 2210 4520 50  0001 C CNN
+F 3 "" H 2210 4520 50  0001 C CNN
+	1    2210 4520
 	1    0    0    -1
 $EndComp
@@
 DIO0
 Text Notes 7000 3680 0    50   ~ 0
-Modulation LoRa\n
+Module LoRa\n
 Text Label 7300 2100 2    50   ~ 0
 DIO0
@@
 DIO5
 NoConn ~ 8700 2000
+$Comp
+L Device:R R?
+U 1 1 5C4A3DDF
+P 720 4230
+F 0 "R?" H 790 4276 50  0000 L CNN
+F 1 "1k" H 790 4185 50  0000 L CNN
+F 2 "" V 650 4230 50  0001 C CNN
+F 3 "~" H 720 4230 50  0001 C CNN
+	1    720  4230
+	1    0    0    -1
+$EndComp
+$Comp
+L Device:LED D?
+U 1 1 5C4A3EFB
+P 720 4650
+F 0 "D?" V 758 4533 50  0000 R CNN
+F 1 "Light ON" V 680 4560 50  0000 R CNN
+F 2 "" H 720 4650 50  0001 C CNN
+F 3 "~" H 720 4650 50  0001 C CNN
+	1    720  4650
+	0    -1   -1   0
+$EndComp
+$Comp
+L Device:C_Small C?
+U 1 1 5C4A4072
+P 1300 4520
+F 0 "C?" H 1392 4566 50  0000 L CNN
+F 1 "0.1uf" H 1392 4475 50  0000 L CNN
+F 2 "" H 1300 4520 50  0001 C CNN
+F 3 "~" H 1300 4520 50  0001 C CNN
+	1    1300 4520
+	1    0    0    -1
+$EndComp
+$Comp
+L Device:R R?
+U 1 1 5C4AE0AA
+P 2680 4130
+F 0 "R?" H 2750 4176 50  0000 L CNN
+F 1 "2.2k" H 2750 4085 50  0000 L CNN
+F 2 "" V 2610 4130 50  0001 C CNN
+F 3 "~" H 2680 4130 50  0001 C CNN
+	1    2680 4130
+	1    0    0    -1
+$EndComp
+$Comp
+L Device:R R?
+U 1 1 5C4AE188
+P 2960 4130
+F 0 "R?" H 3030 4176 50  0000 L CNN
+F 1 "2.2k" H 3030 4085 50  0000 L CNN
+F 2 "" V 2890 4130 50  0001 C CNN
+F 3 "~" H 2960 4130 50  0001 C CNN
+	1    2960 4130
+	1    0    0    -1
+$EndComp
+$Comp
+L power:GND #PWR?
+U 1 1 5C4AE8E4
+P 1300 4700
+F 0 "#PWR?" H 1300 4450 50  0001 C CNN
+F 1 "GND" H 1305 4527 50  0000 C CNN
+F 2 "" H 1300 4700 50  0001 C CNN
+F 3 "" H 1300 4700 50  0001 C CNN
+	1    1300 4700
+	1    0    0    -1
+$EndComp
+$Comp
+L power:GND #PWR?
+U 1 1 5C4AE935
+P 720 4910
+F 0 "#PWR?" H 720 4660 50  0001 C CNN
+F 1 "GND" H 725 4737 50  0000 C CNN
+F 2 "" H 720 4910 50  0001 C CNN
+F 3 "" H 720 4910 50  0001 C CNN
+	1    720  4910
+	1    0    0    -1
+$EndComp
+$Comp
+L power:GND #PWR?
+U 1 1 5C4AE986
+P 1720 4700
+F 0 "#PWR?" H 1720 4450 50  0001 C CNN
+F 1 "GND" H 1725 4527 50  0000 C CNN
+F 2 "" H 1720 4700 50  0001 C CNN
+F 3 "" H 1720 4700 50  0001 C CNN
+	1    1720 4700
+	1    0    0    -1
+$EndComp
+$Comp
+L power:+3.3V #PWR?
+U 1 1 5C4B20BE
+P 720 3990
+F 0 "#PWR?" H 720 3840 50  0001 C CNN
+F 1 "+3.3V" H 735 4163 50  0000 C CNN
+F 2 "" H 720 3990 50  0001 C CNN
+F 3 "" H 720 3990 50  0001 C CNN
+	1    720  3990
+	1    0    0    -1
+$EndComp
+$Comp
+L power:+3.3V #PWR?
+U 1 1 5C4B210F
+P 1300 4320
+F 0 "#PWR?" H 1300 4170 50  0001 C CNN
+F 1 "+3.3V" H 1315 4493 50  0000 C CNN
+F 2 "" H 1300 4320 50  0001 C CNN
+F 3 "" H 1300 4320 50  0001 C CNN
+	1    1300 4320
+	1    0    0    -1
+$EndComp
+$Comp
+L power:+3.3V #PWR?
+U 1 1 5C4B2160
+P 1720 4320
+F 0 "#PWR?" H 1720 4170 50  0001 C CNN
+F 1 "+3.3V" H 1735 4493 50  0000 C CNN
+F 2 "" H 1720 4320 50  0001 C CNN
+F 3 "" H 1720 4320 50  0001 C CNN
+	1    1720 4320
+	1    0    0    -1
+$EndComp
+$Comp
+L power:+3.3V #PWR?
+U 1 1 5C4B21B1
+P 2820 3860
+F 0 "#PWR?" H 2820 3710 50  0001 C CNN
+F 1 "+3.3V" H 2835 4033 50  0000 C CNN
+F 2 "" H 2820 3860 50  0001 C CNN
+F 3 "" H 2820 3860 50  0001 C CNN
+	1    2820 3860
+	1    0    0    -1
+$EndComp
+Text Label 3180 4420 0    50   ~ 0
+SDA
+Text Label 3180 4600 0    50   ~ 0
+SCL
+Text Notes 510  3710 0    50   ~ 0
+Light Sensor
+Wire Wire Line
+	720  3990 720  4080
+Wire Wire Line
+	720  4380 720  4500
+Wire Wire Line
+	720  4800 720  4910
+Wire Wire Line
+	1300 4620 1300 4700
+Wire Wire Line
+	1300 4420 1300 4320
+Wire Wire Line
+	1720 4320 1720 4420
+Wire Wire Line
+	1720 4420 1810 4420
+Wire Wire Line
+	1720 4700 1720 4600
+Wire Wire Line
+	1720 4600 1810 4600
+Wire Wire Line
+	2610 4420 2680 4420
+Wire Wire Line
+	2610 4600 2960 4600
+Wire Wire Line
+	2680 4280 2680 4420
+Connection ~ 2680 4420
+Wire Wire Line
+	2680 4420 3180 4420
+Wire Wire Line
+	2960 4280 2960 4600
+Connection ~ 2960 4600
+Wire Wire Line
+	2960 4600 3180 4600
+Wire Wire Line
+	2960 3980 2960 3860
+Wire Wire Line
+	2960 3860 2820 3860
+Wire Wire Line
+	2680 3980 2680 3860
+Wire Wire Line
+	2680 3860 2820 3860
+Connection ~ 2820 3860
+Text Notes 970  3970 0    50   ~ 0
+7-bit Unshifted I2C Address 0x10
+Wire Notes Line
+	470  5120 3730 5120
+Wire Notes Line
+	3730 5120 3730 3600
 $EndSCHEMATC
