File: Hardware/citizen_sensor.sch (KiCad schematic (older format))
At the start: 35 parts

Commit message: Atmospheric sensor
Parts:
- removed U?: BME280, Package_LGA:Bosch_LGA-8_2.5x2.5mm_P0.65mm_ClockwisePinNumbering, symbol Sensor:BME280
- added C? (x2): 0.1uf, symbol Device:C_Small
- added R? (x3): 4.7K, symbol Device:R
- added U?: BME280, symbol electroniccats:BME280
Connections:
- net labels added: CS_, SDO
- wire segments 123 -> 150
Other:
- note added: "Atmospheric sensor"

Commit message: add sound sensor
Parts:
- removed R? (x2): 2.2k, symbol Device:R
- added C?: 1uf, symbol Device:C_Small
- added R?: 10, symbol Device:R
- added R?: 39, symbol Device:R
- added U?: LM324, symbol Amplifier_Operational:LM324
Changed lines of the file:
@@
 $Descr A4 11693 8268
 encoding utf-8
-Sheet 1 1
+Sheet 1 2
 Title "Citizen_sensor"
 Date ""
@@
 L Connector:Conn_01x02_Female J?
 U 1 1 5C48C861
-P 5030 6830
-F 0 "J?" H 5057 6806 50  0000 L CNN
-F 1 "POM-3044P-R" H 5057 6715 50  0000 L CNN
-F 2 "" H 5030 6830 50  0001 C CNN
-F 3 "~" H 5030 6830 50  0001 C CNN
-	1    5030 6830
+P 4500 7170
+F 0 "J?" H 4527 7146 50  0000 L CNN
+F 1 "POM-3044P-R" H 4527 7055 50  0000 L CNN
+F 2 "" H 4500 7170 50  0001 C CNN
+F 3 "~" H 4500 7170 50  0001 C CNN
+	1    4500 7170
 	1    0    0    -1
 $EndComp
@@
 $EndComp
 $Comp
-L Device:R R?
-U 1 1 5C4AE0AA
-P 2680 4130
-F 0 "R?" H 2750 4176 50  0000 L CNN
-F 1 "2.2k" H 2750 4085 50  0000 L CNN
-F 2 "" V 2610 4130 50  0001 C CNN
-F 3 "~" H 2680 4130 50  0001 C CNN
-	1    2680 4130
-	1    0    0    -1
-$EndComp
-$Comp
-L Device:R R?
-U 1 1 5C4AE188
-P 2960 4130
-F 0 "R?" H 3030 4176 50  0000 L CNN
-F 1 "2.2k" H 3030 4085 50  0000 L CNN
-F 2 "" V 2890 4130 50  0001 C CNN
-F 3 "~" H 2960 4130 50  0001 C CNN
-	1    2960 4130
-	1    0    0    -1
-$EndComp
-$Comp
 L power:GND #PWR?
 U 1 1 5C4AE8E4
@@
 	1    0    0    -1
 $EndComp
-$Comp
-L power:+3.3V #PWR?
-U 1 1 5C4B21B1
-P 2820 3860
-F 0 "#PWR?" H 2820 3710 50  0001 C CNN
-F 1 "+3.3V" H 2835 4033 50  0000 C CNN
-F 2 "" H 2820 3860 50  0001 C CNN
-F 3 "" H 2820 3860 50  0001 C CNN
-	1    2820 3860
-	1    0    0    -1
-$EndComp
 Text Label 3180 4420 0    50   ~ 0
 SDA
@@
 Wire Wire Line
 	2960 4600 3180 4600
-Wire Wire Line
-	2960 3980 2960 3860
-Wire Wire Line
-	2960 3860 2820 3860
-Wire Wire Line
-	2680 3980 2680 3860
-Wire Wire Line
-	2680 3860 2820 3860
-Connection ~ 2820 3860
 Text Notes 970  3970 0    50   ~ 0
 7-bit Unshifted I2C Address 0x10
@@
 Text Label 5100 4440 2    50   ~ 0
 SDO
+$Comp
+L Device:R R?
+U 1 1 5C54F2FC
+P 880 6800
+F 0 "R?" H 950 6846 50  0000 L CNN
+F 1 "10" H 950 6755 50  0000 L CNN
+F 2 "" V 810 6800 50  0001 C CNN
+F 3 "~" H 880 6800 50  0001 C CNN
+	1    880  6800
+	1    0    0    -1
+$EndComp
+$Comp
+L Device:C_Small C?
+U 1 1 5C54F3F8
+P 2860 6770
+F 0 "C?" H 2952 6816 50  0000 L CNN
+F 1 "1uf" H 2952 6725 50  0000 L CNN
+F 2 "" H 2860 6770 50  0001 C CNN
+F 3 "~" H 2860 6770 50  0001 C CNN
+	1    2860 6770
+	1    0    0    -1
+$EndComp
+Wire Wire Line
+	2550 6600 2860 6600
+Wire Wire Line
+	2860 6600 2860 6670
+Wire Wire Line
+	1150 6600 880  6600
+Wire Wire Line
+	880  6600 880  6650
+$Comp
+L power:GND #PWR?
+U 1 1 5C55D89B
+P 880 7010
+F 0 "#PWR?" H 880 6760 50  0001 C CNN
+F 1 "GND" H 885 6837 50  0000 C CNN
+F 2 "" H 880 7010 50  0001 C CNN
+F 3 "" H 880 7010 50  0001 C CNN
+	1    880  7010
+	1    0    0    -1
+$EndComp
+$Comp
+L power:GND #PWR?
+U 1 1 5C55D8FD
+P 2860 6980
+F 0 "#PWR?" H 2860 6730 50  0001 C CNN
+F 1 "GND" H 2865 6807 50  0000 C CNN
+F 2 "" H 2860 6980 50  0001 C CNN
+F 3 "" H 2860 6980 50  0001 C CNN
+	1    2860 6980
+	1    0    0    -1
+$EndComp
+$Comp
+L Device:R R?
+U 1 1 5C55E046
+P 590 6790
+F 0 "R?" H 660 6836 50  0000 L CNN
+F 1 "39" H 660 6745 50  0000 L CNN
+F 2 "" V 520 6790 50  0001 C CNN
+F 3 "~" H 590 6790 50  0001 C CNN
+	1    590  6790
+	1    0    0    -1
+$EndComp
+$Comp
+L Amplifier_Operational:LM324 U?
+U 1 1 5C55E851
+P 4620 6680
+F 0 "U?" H 4620 7047 50  0000 C CNN
+F 1 "LM324" H 4620 6956 50  0000 C CNN
+F 2 "" H 4570 6780 50  0001 C CNN
+F 3 "http://www.ti.com/lit/ds/symlink/lm2902-n.pdf" H 4670 6880 50  0001 C CNN
+	1    4620 6680
+	1    0    0    -1
+$EndComp
+$Sheet
+S 5610 5510 880  180
+U 5C560DC9
+F0 "Sheetsound" 50
+F1 "sensorsound.sch" 50
+$EndSheet
 $EndSCHEMATC

Commit message: sound circuit ampli
Parts:
- removed J?: POM-3044P-R, symbol Connector:Conn_01x02_Female
- removed U?: LM324, symbol Amplifier_Operational:LM324
Changed lines of the file:
@@
-$EndComp
-$Comp
-L Connector:Conn_01x02_Female J?
-U 1 1 5C48C861
-P 4500 7170
-F 0 "J?" H 4527 7146 50  0000 L CNN
-F 1 "POM-3044P-R" H 4527 7055 50  0000 L CNN
-F 2 "" H 4500 7170 50  0001 C CNN
-F 3 "~" H 4500 7170 50  0001 C CNN
-	1    4500 7170
-	1    0    0    -1
 $EndComp
 $Comp
@@
 	1    0    0    -1
 $EndComp
-$Comp
-L Amplifier_Operational:LM324 U?
-U 1 1 5C55E851
-P 4620 6680
-F 0 "U?" H 4620 7047 50  0000 C CNN
-F 1 "LM324" H 4620 6956 50  0000 C CNN
-F 2 "" H 4570 6780 50  0001 C CNN
-F 3 "http://www.ti.com/lit/ds/symlink/lm2902-n.pdf" H 4670 6880 50  0001 C CNN
-	1    4620 6680
-	1    0    0    -1
-$EndComp

Commit message: sensor sound envolvent
Connections:
- wire segments 150 -> 146
Changed lines of the file:
@@
 Wire Wire Line
 	1720 4600 1810 4600
-Wire Wire Line
-	2610 4420 2680 4420
-Wire Wire Line
-	2610 4600 2960 4600
-Wire Wire Line
-	2680 4280 2680 4420
-Connection ~ 2680 4420
-Wire Wire Line
-	2680 4420 3180 4420
-Wire Wire Line
-	2960 4280 2960 4600
-Connection ~ 2960 4600
-Wire Wire Line
-	2960 4600 3180 4600
 Text Notes 970  3970 0    50   ~ 0
 7-bit Unshifted I2C Address 0x10
@@
 F1 "sensorsound.sch" 50
 $EndSheet
+Wire Wire Line
+	2610 4600 3180 4600
+Wire Wire Line
+	2610 4420 3180 4420
 $EndSCHEMATC

Commit message: change VCC with 3.3V sound sensor
Other:
- moved on the sheet: C?, R?
Changed lines of the file:
@@
 L electroniccats:MICS-4514 U?
 U 1 1 5C48BCB3
-P 1850 6500
-F 0 "U?" H 1850 6967 50  0000 C CNN
-F 1 "MICS-4514" H 1850 6876 50  0000 C CNN
-F 2 "MICS_10-SMD" H 1800 6200 50  0001 L BNN
-F 3 "None" H 1800 6200 50  0001 L BNN
-F 4 "None" H 1800 6200 50  0001 L BNN "Field5"
-	1    1850 6500
+P 2300 6090
+F 0 "U?" H 2300 6557 50  0000 C CNN
+F 1 "MICS-4514" H 2300 6466 50  0000 C CNN
+F 2 "MICS_10-SMD" H 2250 5790 50  0001 L BNN
+F 3 "None" H 2250 5790 50  0001 L BNN
+F 4 "None" H 2250 5790 50  0001 L BNN "Field5"
+	1    2300 6090
 	1    0    0    -1
 $EndComp
@@
 L Device:R R?
 U 1 1 5C54F2FC
-P 880 6800
-F 0 "R?" H 950 6846 50  0000 L CNN
-F 1 "10" H 950 6755 50  0000 L CNN
-F 2 "" V 810 6800 50  0001 C CNN
-F 3 "~" H 880 6800 50  0001 C CNN
-	1    880  6800
+P 1330 6390
+F 0 "R?" H 1400 6436 50  0000 L CNN
+F 1 "10" H 1400 6345 50  0000 L CNN
+F 2 "" V 1260 6390 50  0001 C CNN
+F 3 "~" H 1330 6390 50  0001 C CNN
+	1    1330 6390
 	1    0    0    -1
 $EndComp
@@
 L Device:C_Small C?
 U 1 1 5C54F3F8
-P 2860 6770
-F 0 "C?" H 2952 6816 50  0000 L CNN
-F 1 "1uf" H 2952 6725 50  0000 L CNN
-F 2 "" H 2860 6770 50  0001 C CNN
-F 3 "~" H 2860 6770 50  0001 C CNN
-	1    2860 6770
-	1    0    0    -1
-$EndComp
-Wire Wire Line
-	2550 6600 2860 6600
-Wire Wire Line
-	2860 6600 2860 6670
-Wire Wire Line
-	1150 6600 880  6600
-Wire Wire Line
-	880  6600 880  6650
+P 3310 6360
+F 0 "C?" H 3402 6406 50  0000 L CNN
+F 1 "1uf" H 3402 6315 50  0000 L CNN
+F 2 "" H 3310 6360 50  0001 C CNN
+F 3 "~" H 3310 6360 50  0001 C CNN
+	1    3310 6360
+	1    0    0    -1
+$EndComp
+Wire Wire Line
+	3000 6190 3310 6190
+Wire Wire Line
+	3310 6190 3310 6260
+Wire Wire Line
+	1600 6190 1330 6190
+Wire Wire Line
+	1330 6190 1330 6240
 $Comp
 L power:GND #PWR?
 U 1 1 5C55D89B
-P 880 7010
-F 0 "#PWR?" H 880 6760 50  0001 C CNN
-F 1 "GND" H 885 6837 50  0000 C CNN
-F 2 "" H 880 7010 50  0001 C CNN
-F 3 "" H 880 7010 50  0001 C CNN
-	1    880  7010
+P 1330 6600
+F 0 "#PWR?" H 1330 6350 50  0001 C CNN
+F 1 "GND" H 1335 6427 50  0000 C CNN
+F 2 "" H 1330 6600 50  0001 C CNN
+F 3 "" H 1330 6600 50  0001 C CNN
+	1    1330 6600
 	1    0    0    -1
 $EndComp
@@
 L power:GND #PWR?
 U 1 1 5C55D8FD
-P 2860 6980
-F 0 "#PWR?" H 2860 6730 50  0001 C CNN
-F 1 "GND" H 2865 6807 50  0000 C CNN
-F 2 "" H 2860 6980 50  0001 C CNN
-F 3 "" H 2860 6980 50  0001 C CNN
-	1    2860 6980
+P 3310 6570
+F 0 "#PWR?" H 3310 6320 50  0001 C CNN
+F 1 "GND" H 3315 6397 50  0000 C CNN
+F 2 "" H 3310 6570 50  0001 C CNN
+F 3 "" H 3310 6570 50  0001 C CNN
+	1    3310 6570
 	1    0    0    -1
 $EndComp
@@
 L Device:R R?
 U 1 1 5C55E046
-P 590 6790
-F 0 "R?" H 660 6836 50  0000 L CNN
-F 1 "39" H 660 6745 50  0000 L CNN
-F 2 "" V 520 6790 50  0001 C CNN
-F 3 "~" H 590 6790 50  0001 C CNN
-	1    590  6790
+P 1040 6380
+F 0 "R?" H 1110 6426 50  0000 L CNN
+F 1 "39" H 1110 6335 50  0000 L CNN
+F 2 "" V 970 6380 50  0001 C CNN
+F 3 "~" H 1040 6380 50  0001 C CNN
+	1    1040 6380
 	1    0    0    -1
 $EndComp
 $Sheet
-S 5610 5510 880  180
+S 5400 6340 880  180
 U 5C560DC9
 F0 "Sheetsound" 50

Commit message: add capacitor VDDCORE
Parts:
- added C?: 1uf, symbol Device:C_Small
Changed lines of the file:
@@
 L power:GND #PWR?
 U 1 1 5C48F365
-P 9000 1300
-F 0 "#PWR?" H 9000 1050 50  0001 C CNN
-F 1 "GND" H 9005 1127 50  0000 C CNN
-F 2 "" H 9000 1300 50  0001 C CNN
-F 3 "" H 9000 1300 50  0001 C CNN
-	1    9000 1300
+P 8930 1420
+F 0 "#PWR?" H 8930 1170 50  0001 C CNN
+F 1 "GND" H 9060 1340 50  0000 C CNN
+F 2 "" H 8930 1420 50  0001 C CNN
+F 3 "" H 8930 1420 50  0001 C CNN
+	1    8930 1420
 	1    0    0    -1
 $EndComp
@@
 Wire Wire Line
 	9400 1600 9600 1600
-Wire Wire Line
-	8700 1200 9000 1200
-Wire Wire Line
-	9000 1200 9000 1300
 Wire Wire Line
 	7300 1600 7200 1600
@@
 Wire Wire Line
 	2610 4420 3180 4420
+$Comp
+L Device:C_Small C?
+U 1 1 5C61948D
+P 8930 1320
+F 0 "C?" H 9022 1366 50  0000 L CNN
+F 1 "1uf" H 9022 1275 50  0000 L CNN
+F 2 "" H 8930 1320 50  0001 C CNN
+F 3 "~" H 8930 1320 50  0001 C CNN
+	1    8930 1320
+	1    0    0    -1
+$EndComp
+Wire Wire Line
+	8700 1200 8930 1200
+Wire Wire Line
+	8930 1200 8930 1220
 $EndSCHEMATC
