File: Hardware/citizen_sensor.sch (KiCad schematic (older format))
At the start: 39 parts

Commit message: change veml6075 to brakeout
Parts:
- removed C?: 0.1uf, Capacitor_SMD:C_0805_2012Metric_Pad1.15x1.40mm_HandSolder, symbol Device:C_Small
- removed D?: Light ON, symbol Device:LED
- removed R?: 1k, Resistor_SMD:R_0805_2012Metric_Pad1.15x1.40mm_HandSolder, symbol Device:R
- removed U?: VEML6075, symbol electroniccats:VEML6075
- added J?: VEML6075, symbol Connector:Conn_01x04_Female
- D? (x2): footprint (none) -> LED_SMD:LED_0805_2012Metric_Castellated
- R?: value 820 -> 1
- R?: value 820 -> 269
Connections:
- wire segments 151 -> 144
Changed lines of the file:
@@
 F 0 "D?" V 5235 1255 50  0000 C CNN
 F 1 "ON" V 5145 1255 50  0000 C CNN
-F 2 "" H 5220 1105 50  0001 C CNN
+F 2 "LED_SMD:LED_0805_2012Metric_Castellated" H 5220 1105 50  0001 C CNN
 F 3 "~" H 5220 1105 50  0001 C CNN
 	1    5220 1105
@@
 F 3 "~" H 9860 4480 50  0001 C CNN
 	1    9860 4380
-	1    0    0    -1
-$EndComp
-$Comp
-L electroniccats:VEML6075 U?
-U 1 1 5C48D32D
-P 2210 4520
-F 0 "U?" H 2210 4761 50  0000 C CNN
-F 1 "VEML6075" H 2210 4260 50  0000 C CNN
-F 2 "" H 2210 4520 50  0001 C CNN
-F 3 "" H 2210 4520 50  0001 C CNN
-	1    2210 4520
 	1    0    0    -1
 $EndComp
@@
 F 0 "D?" H 2900 2160 50  0000 C CNN
 F 1 "CHARGE" H 2900 2390 50  0000 C CNN
-F 2 "" H 2900 2270 50  0001 C CNN
+F 2 "LED_SMD:LED_0805_2012Metric_Castellated" H 2900 2270 50  0001 C CNN
 F 3 "~" H 2900 2270 50  0001 C CNN
 	1    2900 2270
@@
 NoConn ~ 8700 2000
 $Comp
-L Device:R R?
-U 1 1 5C4A3DDF
-P 720 4230
-F 0 "R?" H 790 4276 50  0000 L CNN
-F 1 "1k" H 790 4185 50  0000 L CNN
-F 2 "Resistor_SMD:R_0805_2012Metric_Pad1.15x1.40mm_HandSolder" V 650 4230 50  0001 C CNN
-F 3 "~" H 720 4230 50  0001 C CNN
-	1    720  4230
-	1    0    0    -1
-$EndComp
-$Comp
-L Device:LED D?
-U 1 1 5C4A3EFB
-P 720 4650
-F 0 "D?" V 758 4533 50  0000 R CNN
-F 1 "Light ON" V 680 4560 50  0000 R CNN
-F 2 "" H 720 4650 50  0001 C CNN
-F 3 "~" H 720 4650 50  0001 C CNN
-	1    720  4650
-	0    -1   -1   0
-$EndComp
-$Comp
-L Device:C_Small C?
-U 1 1 5C4A4072
-P 1300 4520
-F 0 "C?" H 1392 4566 50  0000 L CNN
-F 1 "0.1uf" H 1392 4475 50  0000 L CNN
-F 2 "Capacitor_SMD:C_0805_2012Metric_Pad1.15x1.40mm_HandSolder" H 1300 4520 50  0001 C CNN
-F 3 "~" H 1300 4520 50  0001 C CNN
-	1    1300 4520
-	1    0    0    -1
-$EndComp
-$Comp
-L power:GND #PWR?
-U 1 1 5C4AE8E4
-P 1300 4700
-F 0 "#PWR?" H 1300 4450 50  0001 C CNN
-F 1 "GND" H 1305 4527 50  0000 C CNN
-F 2 "" H 1300 4700 50  0001 C CNN
-F 3 "" H 1300 4700 50  0001 C CNN
-	1    1300 4700
-	1    0    0    -1
-$EndComp
-$Comp
-L power:GND #PWR?
-U 1 1 5C4AE935
-P 720 4910
-F 0 "#PWR?" H 720 4660 50  0001 C CNN
-F 1 "GND" H 725 4737 50  0000 C CNN
-F 2 "" H 720 4910 50  0001 C CNN
-F 3 "" H 720 4910 50  0001 C CNN
-	1    720  4910
-	1    0    0    -1
-$EndComp
-$Comp
 L power:GND #PWR?
 U 1 1 5C4AE986
-P 1720 4700
-F 0 "#PWR?" H 1720 4450 50  0001 C CNN
-F 1 "GND" H 1725 4527 50  0000 C CNN
-F 2 "" H 1720 4700 50  0001 C CNN
-F 3 "" H 1720 4700 50  0001 C CNN
-	1    1720 4700
-	1    0    0    -1
-$EndComp
-$Comp
-L power:+3.3V #PWR?
-U 1 1 5C4B20BE
-P 720 3990
-F 0 "#PWR?" H 720 3840 50  0001 C CNN
-F 1 "+3.3V" H 735 4163 50  0000 C CNN
-F 2 "" H 720 3990 50  0001 C CNN
-F 3 "" H 720 3990 50  0001 C CNN
-	1    720  3990
-	1    0    0    -1
-$EndComp
-$Comp
-L power:+3.3V #PWR?
-U 1 1 5C4B210F
-P 1300 4320
-F 0 "#PWR?" H 1300 4170 50  0001 C CNN
-F 1 "+3.3V" H 1315 4493 50  0000 C CNN
-F 2 "" H 1300 4320 50  0001 C CNN
-F 3 "" H 1300 4320 50  0001 C CNN
-	1    1300 4320
+P 1780 4480
+F 0 "#PWR?" H 1780 4230 50  0001 C CNN
+F 1 "GND" H 1785 4307 50  0000 C CNN
+F 2 "" H 1780 4480 50  0001 C CNN
+F 3 "" H 1780 4480 50  0001 C CNN
+	1    1780 4480
 	1    0    0    -1
 $EndComp
@@
 L power:+3.3V #PWR?
 U 1 1 5C4B2160
-P 1720 4320
-F 0 "#PWR?" H 1720 4170 50  0001 C CNN
-F 1 "+3.3V" H 1735 4493 50  0000 C CNN
-F 2 "" H 1720 4320 50  0001 C CNN
-F 3 "" H 1720 4320 50  0001 C CNN
-	1    1720 4320
-	1    0    0    -1
-$EndComp
-Text Label 3180 4420 0    50   ~ 0
+P 1780 4320
+F 0 "#PWR?" H 1780 4170 50  0001 C CNN
+F 1 "+3.3V" H 1795 4493 50  0000 C CNN
+F 2 "" H 1780 4320 50  0001 C CNN
+F 3 "" H 1780 4320 50  0001 C CNN
+	1    1780 4320
+	1    0    0    -1
+$EndComp
+Text Label 2060 4660 2    50   ~ 0
 SDA
-Text Label 3180 4600 0    50   ~ 0
+Text Label 2060 4560 2    50   ~ 0
 SCL
 Text Notes 510  3710 0    50   ~ 0
 Light Sensor
-Wire Wire Line
-	720  3990 720  4080
-Wire Wire Line
-	720  4380 720  4500
-Wire Wire Line
-	720  4800 720  4910
-Wire Wire Line
-	1300 4620 1300 4700
-Wire Wire Line
-	1300 4420 1300 4320
-Wire Wire Line
-	1720 4320 1720 4420
-Wire Wire Line
-	1720 4420 1810 4420
-Wire Wire Line
-	1720 4700 1720 4600
-Wire Wire Line
-	1720 4600 1810 4600
 Text Notes 970  3970 0    50   ~ 0
 7-bit Unshifted I2C Address 0x10
@@
 P 2880 6290
 F 0 "R?" H 2950 6336 50  0000 L CNN
-F 1 "820" H 2950 6245 50  0000 L CNN
+F 1 "1" H 2950 6245 50  0000 L CNN
 F 2 "" V 2810 6290 50  0001 C CNN
 F 3 "~" H 2880 6290 50  0001 C CNN
@@
 F1 "sensorsound.sch" 50
 $EndSheet
-Wire Wire Line
-	2610 4600 3180 4600
-Wire Wire Line
-	2610 4420 3180 4420
 $Comp
 L Device:C_Small C?
@@
 P 2280 6290
 F 0 "R?" H 2350 6336 50  0000 L CNN
-F 1 "820" H 2350 6245 50  0000 L CNN
+F 1 "269" H 2350 6245 50  0000 L CNN
 F 2 "" V 2210 6290 50  0001 C CNN
 F 3 "~" H 2280 6290 50  0001 C CNN
@@
 Wire Wire Line
 	4160 7180 4260 7180
+$Comp
+L Connector:Conn_01x04_Female J?
+U 1 1 5C56906B
+P 2260 4460
+F 0 "J?" H 2288 4436 50  0000 L CNN
+F 1 "VEML6075" H 2288 4345 50  0000 L CNN
+F 2 "" H 2260 4460 50  0001 C CNN
+F 3 "~" H 2260 4460 50  0001 C CNN
+	1    2260 4460
+	1    0    0    -1
+$EndComp
+Wire Wire Line
+	2060 4360 1780 4360
+Wire Wire Line
+	1780 4360 1780 4320
+Wire Wire Line
+	2060 4460 1780 4460
+Wire Wire Line
+	1780 4460 1780 4480
 $EndSCHEMATC

Commit message: ERC check
Parts:
- removed U?: ATSAMD21E18A-MU, Package_QFP:TQFP-32_7x7mm_P0.8mm, symbol electroniccats:ATSAMD21E18A-MU
- added U8: ATSAMD21E18A-MU, Package_QFP:TQFP-32_7x7mm_P0.8mm, symbol electroniccats:ATSAMD21E18A-MU
- gave numbers to parts that had none: 34
Connections:
- net labels removed: CS_
- wire segments 144 -> 143
- no-connect marks 3 -> 10

Commit message: footprints
Parts:
- J1: footprint (none) -> TerminalBlock_4Ucon:TerminalBlock_4Ucon_1x02_P3.50mm_Vertical
- J3, J4, J5: footprint (none) -> Connector_PinHeader_2.54mm:PinHeader_1x04_P2.54mm_Vertical
- Q1: value Q -> FET
- R1, R2, R3, R4, R6: footprint (none) -> Resistor_SMD:R_0805_2012Metric_Pad1.15x1.40mm_HandSolder
- SW1: footprint (none) -> Button_Switch_SMD:SW_SPST_B3U-1000P
- U1: value TLC272 -> TLC2272; footprint (none) -> Package_SO:SOIC-8_3.9x4.9mm_P1.27mm
Changed lines of the file:
@@
 F 0 "SW1" H 7000 1835 50  0000 C CNN
 F 1 "RST" H 7009 1470 50  0000 C CNN
-F 2 "" H 7000 1600 50  0001 C CNN
+F 2 "Button_Switch_SMD:SW_SPST_B3U-1000P" H 7000 1600 50  0001 C CNN
 F 3 "" H 7000 1600 50  0001 C CNN
 	1    7000 1600
@@
 F 0 "J5" H 10475 2142 50  0000 C CNN
 F 1 "PROG" H 10475 2051 50  0000 C CNN
-F 2 "" H 10425 1925 50  0001 C CNN
+F 2 "Connector_PinHeader_2.54mm:PinHeader_1x04_P2.54mm_Vertical" H 10425 1925 50  0001 C CNN
 F 3 "~" H 10425 1925 50  0001 C CNN
 	1    10425 1925
@@
 F 0 "J1" H 640 2315 50  0000 C CNN
 F 1 "BATT" H 640 2406 50  0000 C CNN
-F 2 "" H 720 2640 50  0001 C CNN
+F 2 "TerminalBlock_4Ucon:TerminalBlock_4Ucon_1x02_P3.50mm_Vertical" H 720 2640 50  0001 C CNN
 F 3 "~" H 720 2640 50  0001 C CNN
 	1    720  2640
@@
 F 0 "R6" H 2950 6336 50  0000 L CNN
 F 1 "1" H 2950 6245 50  0000 L CNN
-F 2 "" V 2810 6290 50  0001 C CNN
+F 2 "Resistor_SMD:R_0805_2012Metric_Pad1.15x1.40mm_HandSolder" V 2810 6290 50  0001 C CNN
 F 3 "~" H 2880 6290 50  0001 C CNN
 	1    2880 6290
@@
 F 0 "R4" H 2650 6336 50  0000 L CNN
 F 1 "30" H 2650 6245 50  0000 L CNN
-F 2 "" V 2510 6290 50  0001 C CNN
+F 2 "Resistor_SMD:R_0805_2012Metric_Pad1.15x1.40mm_HandSolder" V 2510 6290 50  0001 C CNN
 F 3 "~" H 2580 6290 50  0001 C CNN
 	1    2580 6290
@@
 F 0 "J4" H 5618 4116 50  0000 L CNN
 F 1 "BME280" H 5618 4025 50  0000 L CNN
-F 2 "" H 5590 4140 50  0001 C CNN
+F 2 "Connector_PinHeader_2.54mm:PinHeader_1x04_P2.54mm_Vertical" H 5590 4140 50  0001 C CNN
 F 3 "~" H 5590 4140 50  0001 C CNN
 	1    5590 4140
@@
 F 0 "R3" H 2350 6336 50  0000 L CNN
 F 1 "269" H 2350 6245 50  0000 L CNN
-F 2 "" V 2210 6290 50  0001 C CNN
+F 2 "Resistor_SMD:R_0805_2012Metric_Pad1.15x1.40mm_HandSolder" V 2210 6290 50  0001 C CNN
 F 3 "~" H 2280 6290 50  0001 C CNN
 	1    2280 6290
@@
 F 0 "R2" H 2010 6336 50  0000 L CNN
 F 1 "36" H 2010 6245 50  0000 L CNN
-F 2 "" V 1870 6290 50  0001 C CNN
+F 2 "Resistor_SMD:R_0805_2012Metric_Pad1.15x1.40mm_HandSolder" V 1870 6290 50  0001 C CNN
 F 3 "~" H 1940 6290 50  0001 C CNN
 	1    1940 6290
@@
 F 0 "R1" H 2010 5846 50  0000 L CNN
 F 1 "30" H 2010 5755 50  0000 L CNN
-F 2 "" V 1870 5800 50  0001 C CNN
+F 2 "Resistor_SMD:R_0805_2012Metric_Pad1.15x1.40mm_HandSolder" V 1870 5800 50  0001 C CNN
 F 3 "~" H 1940 5800 50  0001 C CNN
 	1    1940 5800
@@
 P 1450 6200
 F 0 "Q1" H 1320 6300 50  0000 L CNN
-F 1 "Q" H 1655 6155 50  0000 L CNN
+F 1 "FET" H 1655 6155 50  0000 L CNN
 F 2 "" H 1650 6300 50  0001 C CNN
 F 3 "~" H 1450 6200 50  0001 C CNN
@@
 P 2230 7200
 F 0 "U1" H 2230 7567 50  0000 C CNN
-F 1 "TLC272" H 2230 7476 50  0000 C CNN
-F 2 "" H 2230 7200 50  0001 C CNN
+F 1 "TLC2272" H 2230 7476 50  0000 C CNN
+F 2 "Package_SO:SOIC-8_3.9x4.9mm_P1.27mm" H 2230 7200 50  0001 C CNN
 F 3 "http://www.ti.com/lit/ds/symlink/tlc272.pdf" H 2230 7200 50  0001 C CNN
 	1    2230 7200
@@
 P 3810 7180
 F 0 "U1" H 3810 7547 50  0000 C CNN
-F 1 "TLC272" H 3810 7456 50  0000 C CNN
-F 2 "" H 3810 7180 50  0001 C CNN
+F 1 "TLC2272" H 3810 7456 50  0000 C CNN
+F 2 "Package_SO:SOIC-8_3.9x4.9mm_P1.27mm" H 3810 7180 50  0001 C CNN
 F 3 "http://www.ti.com/lit/ds/symlink/tlc272.pdf" H 3810 7180 50  0001 C CNN
 	2    3810 7180
@@
 F 0 "J3" H 2288 4436 50  0000 L CNN
 F 1 "VEML6075" H 2288 4345 50  0000 L CNN
-F 2 "" H 2260 4460 50  0001 C CNN
+F 2 "Connector_PinHeader_2.54mm:PinHeader_1x04_P2.54mm_Vertical" H 2260 4460 50  0001 C CNN
 F 3 "~" H 2260 4460 50  0001 C CNN
 	1    2260 4460

Commit message: add fuse
Parts:
- removed Q1: FET, symbol Device:Q_NMOS_DGS
- added F1: Fuse, Fuse:Fuse_1812_4532Metric_Pad1.30x3.40mm_HandSolder, symbol Device:Fuse
- added Q1: 2N7002, symbol Device:Q_NMOS_GSD
- added R20, R?: R, symbol Device:R
- D2, D3: manf# (none) -> APT2012SGC
- J2: manf# (none) -> 629105150521
- U1: manf# (none) -> TLC2272IDR
- U3: manf# (none) -> AP2114H-3.3TRG1
- U8: Field4 ATSAMD21E18A-MU-ND -> (none); Field5 https://www.digikey.com.mx/product-detail/en/microchip-tech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 -> (none); Field6 Microchip -> (none); Field7 ATSAMD21E18A-MU -> (none); Field8 QFN-32 Microchip -> (none); manf# (none) -> ATSAMD21E15B-AUT
Connections:
- wire segments 143 -> 150
Changed lines of the file:
@@
 F 2 "LED_SMD:LED_0805_2012Metric_Castellated" H 5220 1105 50  0001 C CNN
 F 3 "~" H 5220 1105 50  0001 C CNN
+F 4 "APT2012SGC" V 5220 1105 50  0001 C CNN "manf#"
 	1    5220 1105
 	0    -1   -1   0
@@
 L Connector:USB_B J2
 U 1 1 5C48BF75
-P 1400 1300
-F 0 "J2" H 1455 1767 50  0000 C CNN
-F 1 "USB_B_Micro" H 1455 1676 50  0000 C CNN
-F 2 "Connector_USB:USB_Micro-B_Wuerth_629105150521" H 1550 1250 50  0001 C CNN
-F 3 "~" H 1550 1250 50  0001 C CNN
-	1    1400 1300
+P 1075 1295
+F 0 "J2" H 1130 1762 50  0000 C CNN
+F 1 "USB_B_Micro" H 1130 1671 50  0000 C CNN
+F 2 "Connector_USB:USB_Micro-B_Wuerth_629105150521" H 1225 1245 50  0001 C CNN
+F 3 "https://www.mouser.mx/datasheet/2/445/629105150521-469306.pdf" H 1225 1245 50  0001 C CNN
+F 4 "629105150521" H 1075 1295 50  0001 C CNN "manf#"
+	1    1075 1295
 	1    0    0    -1
 $EndComp
@@
 F 1 "AP2114" H 3300 1451 50  0000 C CNN
 F 2 "TO_SOT_Packages_SMD:SOT-223-3_TabPin2" H 3300 1525 50  0001 C CIN
-F 3 "https://www.diodes.com/assets/Datasheets/AP2127.pdf" H 3300 1300 50  0001 C CNN
+F 3 "https://www.mouser.mx/datasheet/2/115/AP2114-271472.pdf" H 3300 1300 50  0001 C CNN
+F 4 "AP2114H-3.3TRG1" H 3300 1300 50  0001 C CNN "manf#"
 	1    3300 1300
 	1    0    0    -1
@@
 L power:VCC #PWR0111
 U 1 1 5C493A4B
-P 1800 900
-F 0 "#PWR0111" H 1800 750 50  0001 C CNN
-F 1 "VCC" H 1817 1073 50  0000 C CNN
-F 2 "" H 1800 900 50  0001 C CNN
-F 3 "" H 1800 900 50  0001 C CNN
-	1    1800 900
+P 1885 890
+F 0 "#PWR0111" H 1885 740 50  0001 C CNN
+F 1 "VCC" H 1902 1063 50  0000 C CNN
+F 2 "" H 1885 890 50  0001 C CNN
+F 3 "" H 1885 890 50  0001 C CNN
+	1    1885 890
 	1    0    0    -1
 $EndComp
@@
 	1    0    0    -1
 $EndComp
-Wire Wire Line
-	1700 1100 1800 1100
-Wire Wire Line
-	1800 1100 1800 900
 $Comp
 L power:GND #PWR0113
 U 1 1 5C4942B1
-P 1300 1800
-F 0 "#PWR0113" H 1300 1550 50  0001 C CNN
-F 1 "GND" H 1305 1627 50  0000 C CNN
-F 2 "" H 1300 1800 50  0001 C CNN
-F 3 "" H 1300 1800 50  0001 C CNN
-	1    1300 1800
-	1    0    0    -1
-$EndComp
-Wire Wire Line
-	1300 1700 1300 1800
-Wire Wire Line
-	1400 1700 1400 1800
-Wire Wire Line
-	1400 1800 1300 1800
-Connection ~ 1300 1800
+P 975 1795
+F 0 "#PWR0113" H 975 1545 50  0001 C CNN
+F 1 "GND" H 980 1622 50  0000 C CNN
+F 2 "" H 975 1795 50  0001 C CNN
+F 3 "" H 975 1795 50  0001 C CNN
+	1    975  1795
+	1    0    0    -1
+$EndComp
+Wire Wire Line
+	975  1695 975  1795
+Wire Wire Line
+	1075 1695 1075 1795
+Wire Wire Line
+	1075 1795 975  1795
+Connection ~ 975  1795
 Text Label 2500 800  0    50   ~ 0
 BATT
@@
 	1    0    0    -1
 $EndComp
-Text Label 1800 1300 0    50   ~ 0
+Text Label 1475 1295 0    50   ~ 0
 D+
-Text Label 1800 1400 0    50   ~ 0
+Text Label 1475 1395 0    50   ~ 0
 D-
 Wire Wire Line
-	1700 1300 1800 1300
-Wire Wire Line
-	1700 1400 1800 1400
+	1375 1295 1475 1295
+Wire Wire Line
+	1375 1395 1475 1395
 Wire Wire Line
 	2200 900  2200 1300
@@
 F 1 "BATT" H 640 2406 50  0000 C CNN
 F 2 "TerminalBlock_4Ucon:TerminalBlock_4Ucon_1x02_P3.50mm_Vertical" H 720 2640 50  0001 C CNN
-F 3 "~" H 720 2640 50  0001 C CNN
+F 3 "" H 720 2640 50  0001 C CNN
 	1    720  2640
 	-1   0    0    1
@@
 F 2 "LED_SMD:LED_0805_2012Metric_Castellated" H 2900 2270 50  0001 C CNN
 F 3 "~" H 2900 2270 50  0001 C CNN
+F 4 "APT2012SGC" H 2900 2270 50  0001 C CNN "manf#"
 	1    2900 2270
 	-1   0    0    1
@@
 $EndComp
 $Comp
-L Device:Q_NMOS_DGS Q1
-U 1 1 5C59F289
-P 1450 6200
-F 0 "Q1" H 1320 6300 50  0000 L CNN
-F 1 "FET" H 1655 6155 50  0000 L CNN
-F 2 "" H 1650 6300 50  0001 C CNN
-F 3 "~" H 1450 6200 50  0001 C CNN
-	1    1450 6200
-	1    0    0    -1
-$EndComp
-$Comp
 L power:GND #PWR0139
 U 1 1 5C5A512E
-P 1550 6500
-F 0 "#PWR0139" H 1550 6250 50  0001 C CNN
-F 1 "GND" H 1555 6327 50  0000 C CNN
-F 2 "" H 1550 6500 50  0001 C CNN
-F 3 "" H 1550 6500 50  0001 C CNN
-	1    1550 6500
-	1    0    0    -1
-$EndComp
-Wire Wire Line
-	1550 6400 1550 6500
-Text Label 1250 6200 2    50   ~ 0
+P 1550 6640
+F 0 "#PWR0139" H 1550 6390 50  0001 C CNN
+F 1 "GND" H 1555 6467 50  0000 C CNN
+F 2 "" H 1550 6640 50  0001 C CNN
+F 3 "" H 1550 6640 50  0001 C CNN
+	1    1550 6640
+	1    0    0    -1
+$EndComp
+Text Label 730  6200 3    50   ~ 0
 PRE_HEALTING
 Wire Wire Line
@@
 F 2 "Package_SO:SOIC-8_3.9x4.9mm_P1.27mm" H 2230 7200 50  0001 C CNN
 F 3 "http://www.ti.com/lit/ds/symlink/tlc272.pdf" H 2230 7200 50  0001 C CNN
+F 4 "TLC2272IDR" H 2230 7200 50  0001 C CNN "manf#"
 	1    2230 7200
 	1    0    0    -1
@@
 F 2 "Package_QFP:TQFP-32_7x7mm_P0.8mm" H 8000 2300 50  0001 L BNN
 F 3 "SAMD21E Series 256 KB Flash 32 KB SRAM 48 MHz 32-Bit Microcontroller - QFN-32" H 8000 2300 50  0001 L BNN
-F 4 "ATSAMD21E18A-MU-ND" H 8000 2300 50  0001 L BNN "Field4"
-F 5 "https://www.digikey.com.mx/product-detail/en/microchip-technology/ATSAMD21E18A-MU/ATSAMD21E18A-MU-ND/4935887?utm_source=snapeda&utm_medium=aggregator&utm_campaign=symbol" H 8000 2300 50  0001 L BNN "Field5"
-F 6 "Microchip" H 8000 2300 50  0001 L BNN "Field6"
-F 7 "ATSAMD21E18A-MU" H 8000 2300 50  0001 L BNN "Field7"
-F 8 "QFN-32 Microchip" H 8000 2300 50  0001 L BNN "Field8"
+F 4 "ATSAMD21E15B-AUT" H 8000 2300 50  0001 C CNN "manf#"
 	1    8000 2300
 	1    0    0    -1
@@
 Wire Wire Line
 	9000 1200 8700 1200
+$Comp
+L Device:Fuse F1
+U 1 1 5C5A4F76
+P 1610 1095
+F 0 "F1" V 1807 1095 50  0000 C CNN
+F 1 "Fuse" V 1716 1095 50  0000 C CNN
+F 2 "Fuse:Fuse_1812_4532Metric_Pad1.30x3.40mm_HandSolder" V 1540 1095 50  0001 C CNN
+F 3 "https://www.mouser.mx/datasheet/2/643/0ZCG_Nov2016-1132141.pdf" H 1610 1095 50  0001 C CNN
+F 4 "0ZCG0030FF2C" V 1610 1095 50  0001 C CNN "manf#"
+	1    1610 1095
+	0    -1   -1   0
+$EndComp
+Wire Wire Line
+	1375 1095 1460 1095
+Wire Wire Line
+	1760 1095 1885 1095
+Wire Wire Line
+	1885 1095 1885 890
+$Comp
+L Device:Q_NMOS_GSD Q1
+U 1 1 5C5BBC9D
+P 1450 6200
+F 0 "Q1" H 1655 6246 50  0000 L CNN
+F 1 "2N7002" H 1205 6370 50  0000 L CNN
+F 2 "" H 1650 6300 50  0001 C CNN
+F 3 "~" H 1450 6200 50  0001 C CNN
+	1    1450 6200
+	1    0    0    -1
+$EndComp
+$Comp
+L Device:R R20
+U 1 1 5C5BCC63
+P 1190 6400
+F 0 "R20" H 1120 6354 50  0000 R CNN
+F 1 "R" H 1120 6445 50  0000 R CNN
+F 2 "" V 1120 6400 50  0001 C CNN
+F 3 "~" H 1190 6400 50  0001 C CNN
+	1    1190 6400
+	-1   0    0    1
+$EndComp
+Wire Wire Line
+	1550 6400 1550 6550
+Wire Wire Line
+	1190 6550 1550 6550
+Connection ~ 1550 6550
+Wire Wire Line
+	1550 6550 1550 6640
+Wire Wire Line
+	1080 6200 1190 6200
+Wire Wire Line
+	1190 6250 1190 6200
+Connection ~ 1190 6200
+Wire Wire Line
+	1190 6200 1250 6200
+$Comp
+L Device:R R?
+U 1 1 5C5EC363
+P 930 6200
+F 0 "R?" V 1137 6200 50  0000 C CNN
+F 1 "R" V 1046 6200 50  0000 C CNN
+F 2 "" V 860 6200 50  0001 C CNN
+F 3 "~" H 930 6200 50  0001 C CNN
+	1    930  6200
+	0    -1   -1   0
+$EndComp
+Wire Wire Line
+	780  6200 730  6200
 $EndSCHEMATC
