File: Hardware/citizen_sensor.sch (KiCad schematic (older format))
At the start: 38 parts, among them J1 BATT, J2 USB_B_Micro, J3 VEML6075, J4 BME280, J5 PROG, Q1 2N7002, SW1 RST, U1 TLC2272, U2 MCP73831, U3 AP2114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

Commit message: add manf# res cap
Parts:
- C1, C2, C4, C5: manf# (none) -> 885012107004
- C10, C8: manf# (none) -> CC0805KKX5R5BB105
- C3, C6, C7, C9: manf# (none) -> 08056C104JAZ2A
- D2: manf# APT2012SGC -> 150080VS75000
- D3: manf# APT2012SGC -> 150080SS75000
- Q1: footprint (none) -> Package_TO_SOT_SMD:SOT-23; manf# (none) -> T2N7002AK,LM
- R1, R4: manf# (none) -> CRCW080530R0FKEAC
- R2: manf# (none) -> ERJ-6ENF36R0V
- R3: manf# (none) -> ESR10EZPJ271
- R5: manf# (none) -> ESR10EZPJ103
- R6: manf# (none) -> RC0805FR-071R
- R7, R8: manf# (none) -> ESR10EZPJ102
- U1: manf# TLC2272IDR -> TLC2272CD
- U1: manf# (none) -> TLC2272CD
- U2: manf# (none) -> MCP73831T-5ACI/OT
- U4: Field5 None -> (none); manf# (none) -> MICS-4514
Connections:
- no-connect marks 10 -> 9
Changed lines of the file:
@@
 F 1 "0.1uf" H 9292 1755 50  0000 L CNN
 F 2 "Capacitor_SMD:C_0805_2012Metric_Pad1.15x1.40mm_HandSolder" H 9200 1800 50  0001 C CNN
-F 3 "~" H 9200 1800 50  0001 C CNN
+F 3 "https://www.mouser.mx/datasheet/2/40/X7RDielectric-777024.pdf" H 9200 1800 50  0001 C CNN
+F 4 "08056C104JAZ2A" H 0   0   50  0001 C CNN "manf#"
 	1    9200 1800
 	1    0    0    -1
@@
 F 1 "ON" V 5145 1255 50  0000 C CNN
 F 2 "LED_SMD:LED_0805_2012Metric_Castellated" H 5220 1105 50  0001 C CNN
-F 3 "~" H 5220 1105 50  0001 C CNN
-F 4 "APT2012SGC" V 5220 1105 50  0001 C CNN "manf#"
+F 3 "https://www.mouser.mx/datasheet/2/445/150080SS75000-368930.pdf" H 5220 1105 50  0001 C CNN
+F 4 "150080SS75000" V 5220 1105 50  0001 C CNN "manf#"
 	1    5220 1105
 	0    -1   -1   0
@@
 F 1 "MICS-4514" H 3770 6166 50  0000 C CNN
 F 2 "MICS_10-SMD" H 3720 5490 50  0001 L BNN
-F 3 "None" H 3720 5490 50  0001 L BNN
-F 4 "None" H 3720 5490 50  0001 L BNN "Field5"
+F 3 "https://www.mouser.mx/datasheet/2/18/0278_Datasheet-MiCS-4514-rev-16-1144833.pdf" H 3720 5490 50  0001 L BNN
+F 4 "MICS-4514" H 0   0   50  0001 C CNN "manf#"
 	1    3770 5790
 	1    0    0    -1
@@
 F 1 "1uf" H 9692 1755 50  0000 L CNN
 F 2 "Capacitor_SMD:C_0805_2012Metric_Pad1.15x1.40mm_HandSolder" H 9600 1800 50  0001 C CNN
-F 3 "~" H 9600 1800 50  0001 C CNN
+F 3 "https://www.mouser.mx/datasheet/2/447/UPY-GPHC_X5R_4V-to-50V_25-1131599.pdf" H 9600 1800 50  0001 C CNN
+F 4 "CC0805KKX5R5BB105" H 0   0   50  0001 C CNN "manf#"
 	1    9600 1800
 	1    0    0    -1
@@
 F 1 "0.1uf" H 6292 1755 50  0000 L CNN
 F 2 "Capacitor_SMD:C_0805_2012Metric_Pad1.15x1.40mm_HandSolder" H 6200 1800 50  0001 C CNN
-F 3 "~" H 6200 1800 50  0001 C CNN
+F 3 "https://www.mouser.mx/datasheet/2/40/X7RDielectric-777024.pdf" H 6200 1800 50  0001 C CNN
+F 4 "08056C104JAZ2A" H 0   0   50  0001 C CNN "manf#"
 	1    6200 1800
 	1    0    0    -1
@@
 F 1 "10uf" H 2792 1455 50  0000 L CNN
 F 2 "Capacitor_SMD:C_0805_2012Metric_Pad1.15x1.40mm_HandSolder" H 2700 1500 50  0001 C CNN
-F 3 "~" H 2700 1500 50  0001 C CNN
+F 3 "https://www.mouser.mx/datasheet/2/445/885012107004-554083.pdf" H 2700 1500 50  0001 C CNN
+F 4 "885012107004" H 2700 1500 50  0001 C CNN "manf#"
 	1    2700 1500
 	1    0    0    -1
@@
 F 1 "0.1uf" H 3892 1455 50  0000 L CNN
 F 2 "Capacitor_SMD:C_0805_2012Metric_Pad1.15x1.40mm_HandSolder" H 3800 1500 50  0001 C CNN
-F 3 "~" H 3800 1500 50  0001 C CNN
+F 3 "https://www.mouser.mx/datasheet/2/40/X7RDielectric-777024.pdf" H 3800 1500 50  0001 C CNN
+F 4 "08056C104JAZ2A" H 0   0   50  0001 C CNN "manf#"
 	1    3800 1500
 	1    0    0    -1
@@
 F 1 "10uf" H 4292 1455 50  0000 L CNN
 F 2 "Capacitor_SMD:C_0805_2012Metric_Pad1.15x1.40mm_HandSolder" H 4200 1500 50  0001 C CNN
-F 3 "~" H 4200 1500 50  0001 C CNN
+F 3 "https://www.mouser.mx/datasheet/2/445/885012107004-554083.pdf" H 4200 1500 50  0001 C CNN
+F 4 "885012107004" H 0   0   50  0001 C CNN "manf#"
 	1    4200 1500
 	1    0    0    -1
@@
 F 1 "1k" H 5290 1435 50  0000 L CNN
 F 2 "Resistor_SMD:R_0805_2012Metric_Pad1.15x1.40mm_HandSolder" V 5150 1480 50  0001 C CNN
-F 3 "~" H 5220 1480 50  0001 C CNN
+F 3 "https://www.mouser.mx/datasheet/2/348/esr-e-1139161.pdf" H 5220 1480 50  0001 C CNN
+F 4 "ESR10EZPJ102" H 0   0   50  0001 C CNN "manf#"
 	1    5220 1480
 	1    0    0    -1
@@
 F 1 "MCP73831" H 3270 3065 50  0000 C CNN
 F 2 "Package_TO_SOT_SMD:SOT-23-5" H 3270 2790 50  0001 C CNN
-F 3 "" H 3270 2790 50  0001 C CNN
+F 3 "https://www.mouser.mx/datasheet/2/268/20001984g-846362.pdf" H 3270 2790 50  0001 C CNN
+F 4 "MCP73831T-5ACI/OT" H 3270 2790 50  0001 C CNN "manf#"
 	1    3270 2790
 	1    0    0    -1
@@
 F 1 "10uf" H 2062 2725 50  0000 L CNN
 F 2 "Capacitor_SMD:C_0805_2012Metric_Pad1.15x1.40mm_HandSolder" H 1970 2770 50  0001 C CNN
-F 3 "~" H 1970 2770 50  0001 C CNN
+F 3 "https://www.mouser.mx/datasheet/2/445/885012107004-554083.pdf" H 1970 2770 50  0001 C CNN
+F 4 "885012107004" H 0   0   50  0001 C CNN "manf#"
 	1    1970 2770
 	1    0    0    -1
@@
 F 1 "10k" V 2770 2790 50  0000 C CNN
 F 2 "Resistor_SMD:R_0805_2012Metric_Pad1.15x1.40mm_HandSolder" V 2620 2790 50  0001 C CNN
-F 3 "~" H 2690 2790 50  0001 C CNN
+F 3 "https://www.mouser.mx/datasheet/2/348/esr-e-1139161.pdf" H 2690 2790 50  0001 C CNN
+F 4 "ESR10EZPJ103" H 0   0   50  0001 C CNN "manf#"
 	1    2690 2790
 	0    1    1    0
@@
 F 1 "10uf" H 3892 2995 50  0000 L CNN
 F 2 "Capacitor_SMD:C_0805_2012Metric_Pad1.15x1.40mm_HandSolder" H 3800 3040 50  0001 C CNN
-F 3 "~" H 3800 3040 50  0001 C CNN
+F 3 "https://www.mouser.mx/datasheet/2/445/885012107004-554083.pdf" H 3800 3040 50  0001 C CNN
+F 4 "885012107004" H 0   0   50  0001 C CNN "manf#"
 	1    3800 3040
 	1    0    0    -1
@@
 F 1 "1k" V 3820 2270 50  0000 C CNN
 F 2 "Resistor_SMD:R_0805_2012Metric_Pad1.15x1.40mm_HandSolder" V 3650 2270 50  0001 C CNN
-F 3 "~" H 3720 2270 50  0001 C CNN
+F 3 "https://www.mouser.mx/datasheet/2/348/esr-e-1139161.pdf" H 3720 2270 50  0001 C CNN
+F 4 "ESR10EZPJ102" H 0   0   50  0001 C CNN "manf#"
 	1    3720 2270
 	0    1    1    0
@@
 F 1 "CHARGE" H 2900 2390 50  0000 C CNN
 F 2 "LED_SMD:LED_0805_2012Metric_Castellated" H 2900 2270 50  0001 C CNN
-F 3 "~" H 2900 2270 50  0001 C CNN
-F 4 "APT2012SGC" H 2900 2270 50  0001 C CNN "manf#"
+F 3 "https://www.mouser.mx/datasheet/2/445/150080VS75000-368934.pdf" H 2900 2270 50  0001 C CNN
+F 4 "150080VS75000" H 2900 2270 50  0001 C CNN "manf#"
 	1    2900 2270
 	-1   0    0    1
@@
 F 1 "0.1uf" H 7872 4945 50  0000 L CNN
 F 2 "Capacitor_SMD:C_0805_2012Metric_Pad1.15x1.40mm_HandSolder" H 7780 4990 50  0001 C CNN
-F 3 "~" H 7780 4990 50  0001 C CNN
+F 3 "https://www.mouser.mx/datasheet/2/40/X7RDielectric-777024.pdf" H 7780 4990 50  0001 C CNN
+F 4 "08056C104JAZ2A" H 0   0   50  0001 C CNN "manf#"
 	1    7780 4990
 	1    0    0    -1
@@
 F 1 "1" H 2950 6245 50  0000 L CNN
 F 2 "Resistor_SMD:R_0805_2012Metric_Pad1.15x1.40mm_HandSolder" V 2810 6290 50  0001 C CNN
-F 3 "~" H 2880 6290 50  0001 C CNN
+F 3 "https://www.mouser.mx/datasheet/2/447/PYu-RC_Group_51_RoHS_L_10-1527934.pdf" H 2880 6290 50  0001 C CNN
+F 4 "RC0805FR-071R" H 0   0   50  0001 C CNN "manf#"
 	1    2880 6290
 	1    0    0    -1
@@
 F 1 "30" H 2650 6245 50  0000 L CNN
 F 2 "Resistor_SMD:R_0805_2012Metric_Pad1.15x1.40mm_HandSolder" V 2510 6290 50  0001 C CNN
-F 3 "~" H 2580 6290 50  0001 C CNN
+F 3 "https://www.mouser.mx/datasheet/2/427/crcwce3-1223726.pdf" H 2580 6290 50  0001 C CNN
+F 4 "CRCW080530R0FKEAC" H 0   0   50  0001 C CNN "manf#"
 	1    2580 6290
 	1    0    0    -1
@@
 F 1 "1uf" H 9092 1295 50  0000 L CNN
 F 2 "Capacitor_SMD:C_0805_2012Metric_Pad1.15x1.40mm_HandSolder" H 9000 1340 50  0001 C CNN
-F 3 "~" H 9000 1340 50  0001 C CNN
+F 3 "https://www.mouser.mx/datasheet/2/447/UPY-GPHC_X5R_4V-to-50V_25-1131599.pdf" H 9000 1340 50  0001 C CNN
+F 4 "CC0805KKX5R5BB105" H 0   0   50  0001 C CNN "manf#"
 	1    9000 1340
 	1    0    0    -1
@@
 F 1 "269" H 2350 6245 50  0000 L CNN
 F 2 "Resistor_SMD:R_0805_2012Metric_Pad1.15x1.40mm_HandSolder" V 2210 6290 50  0001 C CNN
-F 3 "~" H 2280 6290 50  0001 C CNN
+F 3 "https://www.mouser.mx/datasheet/2/348/esr-e-1139161.pdf" H 2280 6290 50  0001 C CNN
+F 4 "ESR10EZPJ271" H 0   0   50  0001 C CNN "manf#"
 	1    2280 6290
 	1    0    0    -1
@@
 F 1 "36" H 2010 6245 50  0000 L CNN
 F 2 "Resistor_SMD:R_0805_2012Metric_Pad1.15x1.40mm_HandSolder" V 1870 6290 50  0001 C CNN
-F 3 "~" H 1940 6290 50  0001 C CNN
+F 3 "https://www.mouser.mx/datasheet/2/315/AOA0000C304-1149620.pdf" H 1940 6290 50  0001 C CNN
+F 4 "ERJ-6ENF36R0V" H 0   0   50  0001 C CNN "manf#"
 	1    1940 6290
 	1    0    0    -1
@@
 F 1 "30" H 2010 5755 50  0000 L CNN
 F 2 "Resistor_SMD:R_0805_2012Metric_Pad1.15x1.40mm_HandSolder" V 1870 5800 50  0001 C CNN
-F 3 "~" H 1940 5800 50  0001 C CNN
+F 3 "https://www.mouser.mx/datasheet/2/427/crcwce3-1223726.pdf" H 1940 5800 50  0001 C CNN
+F 4 "CRCW080530R0FKEAC" H 0   0   50  0001 C CNN "manf#"
 	1    1940 5800
 	1    0    0    -1
@@
 F 1 "TLC2272" H 2230 7476 50  0000 C CNN
 F 2 "Package_SO:SOIC-8_3.9x4.9mm_P1.27mm" H 2230 7200 50  0001 C CNN
-F 3 "http://www.ti.com/lit/ds/symlink/tlc272.pdf" H 2230 7200 50  0001 C CNN
-F 4 "TLC2272IDR" H 2230 7200 50  0001 C CNN "manf#"
+F 3 "http://www.ti.com/lit/ds/symlink/tlc2272.pdf" H 2230 7200 50  0001 C CNN
+F 4 "TLC2272CD" H 2230 7200 50  0001 C CNN "manf#"
 	1    2230 7200
 	1    0    0    -1
@@
 F 1 "TLC2272" H 3810 7456 50  0000 C CNN
 F 2 "Package_SO:SOIC-8_3.9x4.9mm_P1.27mm" H 3810 7180 50  0001 C CNN
-F 3 "http://www.ti.com/lit/ds/symlink/tlc272.pdf" H 3810 7180 50  0001 C CNN
+F 3 "http://www.ti.com/lit/ds/symlink/tlc2272.pdf" H 3810 7180 50  0001 C CNN
+F 4 "TLC2272CD" H 0   0   50  0001 C CNN "manf#"
 	2    3810 7180
 	1    0    0    -1
@@
 Connection ~ 3800 1300
 NoConn ~ 7300 2600
-NoConn ~ 4415 6230
 Wire Wire Line
 	9000 1240 9000 1200
@@
 F 0 "Q1" H 1655 6246 50  0000 L CNN
 F 1 "2N7002" H 1205 6370 50  0000 L CNN
-F 2 "" H 1650 6300 50  0001 C CNN
-F 3 "~" H 1450 6200 50  0001 C CNN
+F 2 "Package_TO_SOT_SMD:SOT-23" H 1650 6300 50  0001 C CNN
+F 3 "https://www.mouser.mx/datasheet/2/408/T2N7002AK_datasheet_en_20150401-708738.pdf" H 1450 6200 50  0001 C CNN
+F 4 "T2N7002AK,LM" H 0   0   50  0001 C CNN "manf#"
 	1    1450 6200
 	1    0    0    -1

Commit message: BOM file .csv
Parts:
- AE1: manf# (none) -> 977325
- D1: footprint (none) -> Diode_SMD:D_SOD-123; manf# (none) -> NRVB120VLSFT1G
- J1: manf# (none) -> 1751248
- R20: value R -> 66.5k; footprint (none) -> Resistor_SMD:R_0805_2012Metric_Pad1.15x1.40mm_HandSolder; manf# (none) -> ERJ-6ENF6652V
- R21: renamed from R?; value R -> 66.5; footprint (none) -> Resistor_SMD:R_0805_2012Metric_Pad1.15x1.40mm_HandSolder; manf# (none) -> CRCW080566R5FKEA
- SW1: footprint Button_Switch_SMD:SW_SPST_B3U-1000P -> Button_Switch_SMD:SW_SPST_TL3342; manf# (none) -> DC12V 4 Pins
- U6: manf# (none) -> RFM95W
Changed lines of the file:
@@
 F 0 "SW1" H 7000 1835 50  0000 C CNN
 F 1 "RST" H 7009 1470 50  0000 C CNN
-F 2 "Button_Switch_SMD:SW_SPST_B3U-1000P" H 7000 1600 50  0001 C CNN
-F 3 "" H 7000 1600 50  0001 C CNN
+F 2 "Button_Switch_SMD:SW_SPST_TL3342" H 7000 1600 50  0001 C CNN
+F 3 "https://www.banggood.com/1000Pcs-DC12V-4-Pins-Tact-Tactile-Push-Button-Switch-Momentary-SMD-Switch-5x5x1_5MM-p-1297259.html?rmmds=newArrivals&cur_warehouse=CN" H 7000 1600 50  0001 C CNN
+F 4 "DC12V 4 Pins" H 0   0   50  0001 C CNN "manf#"
 	1    7000 1600
 	1    0    0    -1
@@
 F 1 "RFM95W-868S2" H 8590 4400 50  0000 C CNN
 F 2 "Rf:RFM95W" H 5780 6650 50  0001 C CNN
-F 3 "http://www.hoperf.com/upload/rf/RFM95_96_97_98W.pdf" H 5780 6650 50  0001 C CNN
+F 3 "~" H 5780 6650 50  0001 C CNN
+F 4 "RFM95W" H 0   0   50  0001 C CNN "manf#"
 	1    9080 5000
 	1    0    0    -1
@@
 F 1 "Antenna_Shield" H 10000 4330 50  0000 L CNN
 F 2 "Rf:AMPHENOL_901-144" H 9860 4480 50  0001 C CNN
-F 3 "~" H 9860 4480 50  0001 C CNN
+F 3 "https://www.banggood.com/2pcs-RP-SMA-Female-Adapter-PCB-Edge-Mount-Solder-RF-Connector-p-977325.html?akmClientCountry=MX&&cur_warehouse=CN" H 9860 4480 50  0001 C CNN
+F 4 "977325" H 0   0   50  0001 C CNN "manf#"
 	1    9860 4380
 	1    0    0    -1
@@
 F 2 "Connector_PinHeader_2.54mm:PinHeader_1x04_P2.54mm_Vertical" H 10425 1925 50  0001 C CNN
 F 3 "~" H 10425 1925 50  0001 C CNN
+F 4 "~" H 0   0   50  0001 C CNN "manf#"
 	1    10425 1925
 	1    0    0    -1
@@
 Wire Wire Line
 	2700 1400 2700 1300
-Connection ~ 2700 1300
-Wire Wire Line
-	2700 1300 3000 1300
 Wire Wire Line
 	2700 1600 2700 1800
@@
 F 0 "D1" V 2546 971 50  0000 R CNN
 F 1 "D_Schottky" V 2455 971 50  0000 R CNN
-F 2 "" H 2500 1050 50  0001 C CNN
-F 3 "~" H 2500 1050 50  0001 C CNN
+F 2 "Diode_SMD:D_SOD-123" H 2500 1050 50  0001 C CNN
+F 3 "https://www.mouser.mx/datasheet/2/308/MBR120VLSFT1-D-1074021.pdf" H 2500 1050 50  0001 C CNN
+F 4 "NRVB120VLSFT1G" V 2500 1050 50  0001 C CNN "manf#"
 	1    2500 1050
 	0    -1   -1   0
@@
 F 1 "BATT" H 640 2406 50  0000 C CNN
 F 2 "TerminalBlock_4Ucon:TerminalBlock_4Ucon_1x02_P3.50mm_Vertical" H 720 2640 50  0001 C CNN
-F 3 "" H 720 2640 50  0001 C CNN
+F 3 "https://www.mouser.mx/datasheet/2/324/ItemDetail_1751248-916542.pdf" H 720 2640 50  0001 C CNN
+F 4 "1751248" H 0   0   50  0001 C CNN "manf#"
 	1    720  2640
 	-1   0    0    1
@@
 	2920 2640 2510 2640
 Wire Wire Line
-	1660 2640 1660 2610
-Wire Wire Line
 	1970 2670 1970 2640
-Connection ~ 1970 2640
 $Comp
 L power:GND #PWR0122
@@
 SDO- GND ADDRESS 0X76\nSDO- VDIO ADDRESS 0X77\n\n\n
 Wire Wire Line
-	1660 2640 1970 2640
-Wire Wire Line
 	1970 2870 1970 2970
 Wire Wire Line
@@
 F 2 "Connector_PinHeader_2.54mm:PinHeader_1x04_P2.54mm_Vertical" H 5590 4140 50  0001 C CNN
 F 3 "~" H 5590 4140 50  0001 C CNN
+F 4 "~" H 0   0   50  0001 C CNN "manf#"
 	1    5590 4140
 	1    0    0    -1
@@
 F 2 "Connector_PinHeader_2.54mm:PinHeader_1x04_P2.54mm_Vertical" H 2260 4460 50  0001 C CNN
 F 3 "~" H 2260 4460 50  0001 C CNN
+F 4 "~" H 0   0   50  0001 C CNN "manf#"
 	1    2260 4460
 	1    0    0    -1
@@
 P 1190 6400
 F 0 "R20" H 1120 6354 50  0000 R CNN
-F 1 "R" H 1120 6445 50  0000 R CNN
-F 2 "" V 1120 6400 50  0001 C CNN
-F 3 "~" H 1190 6400 50  0001 C CNN
+F 1 "66.5k" H 1120 6445 50  0000 R CNN
+F 2 "Resistor_SMD:R_0805_2012Metric_Pad1.15x1.40mm_HandSolder" V 1120 6400 50  0001 C CNN
+F 3 "https://www.mouser.mx/datasheet/2/315/AOA0000C304-1149620.pdf" H 1190 6400 50  0001 C CNN
+F 4 "ERJ-6ENF6652V" H 0   0   50  0001 C CNN "manf#"
 	1    1190 6400
 	-1   0    0    1
@@
 	1190 6200 1250 6200
 $Comp
-L Device:R R?
+L Device:R R21
 U 1 1 5C5EC363
 P 930 6200
-F 0 "R?" V 1137 6200 50  0000 C CNN
-F 1 "R" V 1046 6200 50  0000 C CNN
-F 2 "" V 860 6200 50  0001 C CNN
-F 3 "~" H 930 6200 50  0001 C CNN
+F 0 "R21" V 1137 6200 50  0000 C CNN
+F 1 "66.5" V 1046 6200 50  0000 C CNN
+F 2 "Resistor_SMD:R_0805_2012Metric_Pad1.15x1.40mm_HandSolder" V 860 6200 50  0001 C CNN
+F 3 "https://www.mouser.mx/datasheet/2/427/dcrcwe3-109170.pdf" H 930 6200 50  0001 C CNN
+F 4 "CRCW080566R5FKEA" H 0   0   50  0001 C CNN "manf#"
 	1    930  6200
 	0    -1   -1   0
@@
 Wire Wire Line
 	780  6200 730  6200
+Wire Wire Line
+	3000 1300 2700 1300
+Connection ~ 2700 1300
+Wire Wire Line
+	1660 2610 1660 2640
+Wire Wire Line
+	1660 2640 1970 2640
+Connection ~ 1970 2640
 $EndSCHEMATC

Commit message: footprint mics4514
Parts:
- U4: footprint MICS_10-SMD -> MICS-4514:MICS_10-SMD
Changed lines of the file:
@@
 F 0 "U4" H 3770 6257 50  0000 C CNN
 F 1 "MICS-4514" H 3770 6166 50  0000 C CNN
-F 2 "MICS_10-SMD" H 3720 5490 50  0001 L BNN
+F 2 "MICS-4514:MICS_10-SMD" H 3720 5490 50  0001 L BNN
 F 3 "https://www.mouser.mx/datasheet/2/18/0278_Datasheet-MiCS-4514-rev-16-1144833.pdf" H 3720 5490 50  0001 L BNN
 F 4 "MICS-4514" H 0   0   50  0001 C CNN "manf#"

Commit message: add css811
Parts:
- added J?: CSS811, symbol Connector:Conn_01x08_Female
Connections:
- net labels added: INTCSS, RESET, WAKE
- wire segments 150 -> 154
- no-connect marks 9 -> 8
Other:
- note added: "7-bit Unshifted \nI2C Address 0x10"
- note added: "Air quality CSS811"
- note removed: "7-bit Unshifted I2C Address 0x10"
Changed lines of the file:
@@
 L power:GND #PWR0130
 U 1 1 5C4AE986
-P 1780 4480
-F 0 "#PWR0130" H 1780 4230 50  0001 C CNN
-F 1 "GND" H 1785 4307 50  0000 C CNN
-F 2 "" H 1780 4480 50  0001 C CNN
-F 3 "" H 1780 4480 50  0001 C CNN
-	1    1780 4480
+P 600 4430
+F 0 "#PWR0130" H 600 4180 50  0001 C CNN
+F 1 "GND" H 605 4257 50  0000 C CNN
+F 2 "" H 600 4430 50  0001 C CNN
+F 3 "" H 600 4430 50  0001 C CNN
+	1    600  4430
 	1    0    0    -1
 $EndComp
@@
 L power:+3.3V #PWR0131
 U 1 1 5C4B2160
-P 1780 4320
-F 0 "#PWR0131" H 1780 4170 50  0001 C CNN
-F 1 "+3.3V" H 1795 4493 50  0000 C CNN
-F 2 "" H 1780 4320 50  0001 C CNN
-F 3 "" H 1780 4320 50  0001 C CNN
-	1    1780 4320
-	1    0    0    -1
-$EndComp
-Text Label 2060 4660 2    50   ~ 0
+P 600 4270
+F 0 "#PWR0131" H 600 4120 50  0001 C CNN
+F 1 "+3.3V" H 615 4443 50  0000 C CNN
+F 2 "" H 600 4270 50  0001 C CNN
+F 3 "" H 600 4270 50  0001 C CNN
+	1    600  4270
+	1    0    0    -1
+$EndComp
+Text Label 880  4610 2    50   ~ 0
 SDA
-Text Label 2060 4560 2    50   ~ 0
+Text Label 880  4510 2    50   ~ 0
 SCL
 Text Notes 510  3710 0    50   ~ 0
 Light Sensor
-Text Notes 970  3970 0    50   ~ 0
-7-bit Unshifted I2C Address 0x10
+Text Notes 570  4980 0    50   ~ 0
+7-bit Unshifted \nI2C Address 0x10
 Wire Notes Line
-	3730 5120 3730 3600
-Text Notes 3760 3690 0    50   ~ 0
+	1570 5120 1570 3600
+Text Notes 1590 3700 0    50   ~ 0
 Atmospheric sensor
 Wire Notes Line
 	470  5120 6970 5120
-Text Label 5390 4340 2    50   ~ 0
+Text Label 2140 4410 2    50   ~ 0
 SDA
-Text Label 5390 4240 2    50   ~ 0
+Text Label 2140 4310 2    50   ~ 0
 SCL
 $Comp
 L power:+3.3V #PWR0132
 U 1 1 5C535856
-P 5120 3960
-F 0 "#PWR0132" H 5120 3810 50  0001 C CNN
-F 1 "+3.3V" H 5280 4010 50  0000 C CNN
-F 2 "" H 5120 3960 50  0001 C CNN
-F 3 "" H 5120 3960 50  0001 C CNN
-	1    5120 3960
+P 1870 4030
+F 0 "#PWR0132" H 1870 3880 50  0001 C CNN
+F 1 "+3.3V" H 2030 4080 50  0000 C CNN
+F 2 "" H 1870 4030 50  0001 C CNN
+F 3 "" H 1870 4030 50  0001 C CNN
+	1    1870 4030
 	1    0    0    -1
 $EndComp
@@
 Text GLabel 7260 1970 0    50   Input ~ 0
 ENVOL
-Text Notes 4900 4900 0    50   ~ 0
+Text Notes 1650 4970 0    50   ~ 0
 SDO- GND ADDRESS 0X76\nSDO- VDIO ADDRESS 0X77\n\n\n
 Wire Wire Line
@@
 L Connector:Conn_01x04_Female J4
 U 1 1 5C547954
-P 5590 4140
-F 0 "J4" H 5618 4116 50  0000 L CNN
-F 1 "BME280" H 5618 4025 50  0000 L CNN
-F 2 "Connector_PinHeader_2.54mm:PinHeader_1x04_P2.54mm_Vertical" H 5590 4140 50  0001 C CNN
-F 3 "~" H 5590 4140 50  0001 C CNN
-F 4 "~" H 0   0   50  0001 C CNN "manf#"
-	1    5590 4140
+P 2340 4210
+F 0 "J4" H 2368 4186 50  0000 L CNN
+F 1 "BME280" H 2368 4095 50  0000 L CNN
+F 2 "Connector_PinHeader_2.54mm:PinHeader_1x04_P2.54mm_Vertical" H 2340 4210 50  0001 C CNN
+F 3 "~" H 2340 4210 50  0001 C CNN
+F 4 "~" H -3250 70  50  0001 C CNN "manf#"
+	1    2340 4210
 	1    0    0    -1
 $EndComp
@@
 L power:GND #PWR0133
 U 1 1 5C54CAD9
-P 5120 4170
-F 0 "#PWR0133" H 5120 3920 50  0001 C CNN
-F 1 "GND" H 5125 3997 50  0000 C CNN
-F 2 "" H 5120 4170 50  0001 C CNN
-F 3 "" H 5120 4170 50  0001 C CNN
-	1    5120 4170
-	1    0    0    -1
-$EndComp
-Wire Wire Line
-	5390 4140 5120 4140
-Wire Wire Line
-	5120 4140 5120 4170
-Wire Wire Line
-	5120 3960 5120 4040
-Wire Wire Line
-	5120 4040 5390 4040
+P 1870 4240
+F 0 "#PWR0133" H 1870 3990 50  0001 C CNN
+F 1 "GND" H 1875 4067 50  0000 C CNN
+F 2 "" H 1870 4240 50  0001 C CNN
+F 3 "" H 1870 4240 50  0001 C CNN
+	1    1870 4240
+	1    0    0    -1
+$EndComp
+Wire Wire Line
+	2140 4210 1870 4210
+Wire Wire Line
+	1870 4210 1870 4240
+Wire Wire Line
+	1870 4030 1870 4110
+Wire Wire Line
+	1870 4110 2140 4110
 $Comp
 L power:+3.3V #PWR0134
@@
 L Connector:Conn_01x04_Female J3
 U 1 1 5C56906B
-P 2260 4460
-F 0 "J3" H 2288 4436 50  0000 L CNN
-F 1 "VEML6075" H 2288 4345 50  0000 L CNN
-F 2 "Connector_PinHeader_2.54mm:PinHeader_1x04_P2.54mm_Vertical" H 2260 4460 50  0001 C CNN
-F 3 "~" H 2260 4460 50  0001 C CNN
-F 4 "~" H 0   0   50  0001 C CNN "manf#"
-	1    2260 4460
-	1    0    0    -1
-$EndComp
-Wire Wire Line
-	2060 4360 1780 4360
-Wire Wire Line
-	1780 4360 1780 4320
-Wire Wire Line
-	2060 4460 1780 4460
-Wire Wire Line
-	1780 4460 1780 4480
-NoConn ~ 7300 2400
-NoConn ~ 7300 2500
+P 1080 4410
+F 0 "J3" H 1108 4386 50  0000 L CNN
+F 1 "VEML6075" H 1108 4295 50  0000 L CNN
+F 2 "Connector_PinHeader_2.54mm:PinHeader_1x04_P2.54mm_Vertical" H 1080 4410 50  0001 C CNN
+F 3 "~" H 1080 4410 50  0001 C CNN
+F 4 "~" H -1180 -50 50  0001 C CNN "manf#"
+	1    1080 4410
+	1    0    0    -1
+$EndComp
+Wire Wire Line
+	880  4310 600  4310
+Wire Wire Line
+	600  4310 600  4270
+Wire Wire Line
+	880  4410 600  4410
+Wire Wire Line
+	600  4410 600  4430
 NoConn ~ 7300 2800
 NoConn ~ 7300 2900
@@
 	1660 2640 1970 2640
 Connection ~ 1970 2640
+Wire Notes Line
+	2760 3600 2760 5120
+Text Notes 2840 3700 0    50   ~ 0
+Air quality CSS811
+$Comp
+L Connector:Conn_01x08_Female J?
+U 1 1 5C6DC748
+P 3590 4230
+F 0 "J?" H 3617 4206 50  0000 L CNN
+F 1 "CSS811" H 3617 4115 50  0000 L CNN
+F 2 "" H 3590 4230 50  0001 C CNN
+F 3 "~" H 3590 4230 50  0001 C CNN
+	1    3590 4230
+	1    0    0    -1
+$EndComp
+$Comp
+L power:+3.3V #PWR?
+U 1 1 5C6DD8A6
+P 3060 3880
+F 0 "#PWR?" H 3060 3730 50  0001 C CNN
+F 1 "+3.3V" H 3220 3930 50  0000 C CNN
+F 2 "" H 3060 3880 50  0001 C CNN
+F 3 "" H 3060 3880 50  0001 C CNN
+	1    3060 3880
+	1    0    0    -1
+$EndComp
+$Comp
+L power:GND #PWR?
+U 1 1 5C6DD901
+P 3060 4060
+F 0 "#PWR?" H 3060 3810 50  0001 C CNN
+F 1 "GND" H 3065 3887 50  0000 C CNN
+F 2 "" H 3060 4060 50  0001 C CNN
+F 3 "" H 3060 4060 50  0001 C CNN
+	1    3060 4060
+	1    0    0    -1
+$EndComp
+Text Label 3390 4130 2    50   ~ 0
+SCL
+Text Label 3390 4230 2    50   ~ 0
+SDA
+Text Label 3390 4330 2    50   ~ 0
+WAKE
+Text Label 3390 4430 2    50   ~ 0
+INTCSS
+Text Label 3390 4530 2    50   ~ 0
+RESET
+Text Label 6700 1600 2    50   ~ 0
+RESET
+NoConn ~ 3390 4630
+Wire Wire Line
+	3390 3930 3060 3930
+Wire Wire Line
+	3060 3930 3060 3880
+Wire Wire Line
+	3390 4030 3060 4030
+Wire Wire Line
+	3060 4030 3060 4060
+Wire Notes Line
+	4030 3600 4030 5120
+Text Label 7300 2500 2    50   ~ 0
+INTCSS
+Text Label 7300 2400 2    50   ~ 0
+WAKE
 $EndSCHEMATC
