File: Hardware/citizen_sensor.sch (KiCad schematic (older format))
At the start: 39 parts, among them J1 BATT, J2 USB_B_Micro, J3 VEML6075, J4 BME280, J5 PROG, Q1 2N7002, SW1 RST, U1 TLC2272, U2 MCP73831, U3 AP2114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

Commit message: voltaje divisor batt level
Parts:
- added C16: 0.1uf, Capacitor_SMD:C_0805_2012Metric_Pad1.15x1.40mm_HandSolder, symbol Device:C_Small
- added J7: MAX30105, Connector_PinHeader_2.54mm:PinHeader_1x05_P2.54mm_Vertical, symbol Connector:Conn_01x05_Female
- added R22: 680k, Resistor_SMD:R_0805_2012Metric_Pad1.15x1.40mm_HandSolder, symbol Device:R
- added R23: 330k, Resistor_SMD:R_0805_2012Metric_Pad1.15x1.40mm_HandSolder, symbol Device:R
- J6: renamed from J?; footprint (none) -> Connector_PinHeader_2.54mm:PinHeader_1x08_P2.54mm_Vertical; manf# (none) -> -
Connections:
- net labels added: BATTLEVEL, INT
- wire segments 154 -> 166
- no-connect marks 8 -> 6
Other:
- note added: "Smoke sensor"
- note added: "Temperature, \nhumidity and pression"
- note removed: "Atmospheric sensor"
- moved on the sheet: J3, J4, J6

Commit message: PCB read net list
Parts:
- U3: footprint TO_SOT_Packages_SMD:SOT-223-3_TabPin2 -> Package_TO_SOT_SMD:SOT-223-3_TabPin2
- U4: footprint MICS-4514:MICS_10-SMD -> MICS4514:MICS_10-SMD
Changed lines of the file:
@@
 F 0 "U4" H 3770 6257 50  0000 C CNN
 F 1 "MICS-4514" H 3770 6166 50  0000 C CNN
-F 2 "MICS-4514:MICS_10-SMD" H 3720 5490 50  0001 L BNN
+F 2 "MICS4514:MICS_10-SMD" H 3720 5490 50  0001 L BNN
 F 3 "https://www.mouser.mx/datasheet/2/18/0278_Datasheet-MiCS-4514-rev-16-1144833.pdf" H 3720 5490 50  0001 L BNN
 F 4 "MICS-4514" H 0   0   50  0001 C CNN "manf#"
@@
 F 0 "U3" H 3300 1542 50  0000 C CNN
 F 1 "AP2114" H 3300 1451 50  0000 C CNN
-F 2 "TO_SOT_Packages_SMD:SOT-223-3_TabPin2" H 3300 1525 50  0001 C CIN
+F 2 "Package_TO_SOT_SMD:SOT-223-3_TabPin2" H 3300 1525 50  0001 C CIN
 F 3 "https://www.mouser.mx/datasheet/2/115/AP2114-271472.pdf" H 3300 1300 50  0001 C CNN
 F 4 "AP2114H-3.3TRG1" H 3300 1300 50  0001 C CNN "manf#"

Commit message: Update schematic
Parts:
- U2: symbol electroniccats:MCP73831 -> citizen_sensor-rescue:MCP73831-electroniccats
- U4: symbol electroniccats:MICS-4514 -> citizen_sensor-rescue:MICS-4514-electroniccats
- U8: symbol electroniccats:ATSAMD21E18A-MU -> citizen_sensor-rescue:ATSAMD21E18A-MU-electroniccats; manf# ATSAMD21E15B-AUT -> ATSAMD21E18A-AUT
Changed lines of the file:
@@
 $EndComp
 $Comp
-L electroniccats:MICS-4514 U4
+L citizen_sensor-rescue:MICS-4514-electroniccats U4
 U 1 1 5C48BCB3
 P 3770 5790
@@
 	2500 800  2500 900
 $Comp
-L electroniccats:MCP73831 U2
+L citizen_sensor-rescue:MCP73831-electroniccats U2
 U 1 1 5C49572E
 P 3270 2790
@@
 	4620 5590 4620 5690
 $Comp
-L electroniccats:ATSAMD21E18A-MU U8
+L citizen_sensor-rescue:ATSAMD21E18A-MU-electroniccats U8
 U 1 1 5C5C9AE3
 P 8000 2300
@@
 F 2 "Package_QFP:TQFP-32_7x7mm_P0.8mm" H 8000 2300 50  0001 L BNN
 F 3 "SAMD21E Series 256 KB Flash 32 KB SRAM 48 MHz 32-Bit Microcontroller - QFN-32" H 8000 2300 50  0001 L BNN
-F 4 "ATSAMD21E15B-AUT" H 8000 2300 50  0001 C CNN "manf#"
+F 4 "ATSAMD21E18A-AUT" H 8000 2300 50  0001 C CNN "manf#"
 	1    8000 2300
 	1    0    0    -1

Commit message: fix VDD y GND of TLC2272
Parts:
- removed U1: TLC2272, Package_SO:SOIC-8_3.9x4.9mm_P1.27mm, symbol Amplifier_Operational:TLC272
- added U1: TLC2272, Package_SO:SOIC-8_3.9x4.9mm_P1.27mm, symbol Amplifier_Operational:OPA1602
- U2: symbol citizen_sensor-rescue:MCP73831-electroniccats -> citizen_sensor-rescue:MCP73831-electroniccats-citizen_sensor-rescue
- U4: symbol citizen_sensor-rescue:MICS-4514-electroniccats -> citizen_sensor-rescue:MICS-4514-electroniccats-citizen_sensor-rescue
- U8: symbol citizen_sensor-rescue:ATSAMD21E18A-MU-electroniccats -> citizen_sensor-rescue:ATSAMD21E18A-MU-electroniccats-citizen_sensor-rescue
Changed lines of the file:
@@
 $EndComp
 $Comp
-L citizen_sensor-rescue:MICS-4514-electroniccats U4
+L citizen_sensor-rescue:MICS-4514-electroniccats-citizen_sensor-rescue U4
 U 1 1 5C48BCB3
 P 3770 5790
@@
 	2500 800  2500 900
 $Comp
-L citizen_sensor-rescue:MCP73831-electroniccats U2
+L citizen_sensor-rescue:MCP73831-electroniccats-citizen_sensor-rescue U2
 U 1 1 5C49572E
 P 3270 2790
@@
 Text Label 7300 2300 2    50   ~ 0
 ADC_RED
-$Comp
-L Amplifier_Operational:TLC272 U1
-U 1 1 5C64EF5E
-P 2230 7200
-F 0 "U1" H 2230 7567 50  0000 C CNN
-F 1 "TLC2272" H 2230 7476 50  0000 C CNN
-F 2 "Package_SO:SOIC-8_3.9x4.9mm_P1.27mm" H 2230 7200 50  0001 C CNN
-F 3 "http://www.ti.com/lit/ds/symlink/tlc2272.pdf" H 2230 7200 50  0001 C CNN
-F 4 "TLC2272CD" H 2230 7200 50  0001 C CNN "manf#"
-	1    2230 7200
-	1    0    0    -1
-$EndComp
-$Comp
-L Amplifier_Operational:TLC272 U1
-U 2 1 5C655037
-P 3810 7180
-F 0 "U1" H 3810 7547 50  0000 C CNN
-F 1 "TLC2272" H 3810 7456 50  0000 C CNN
-F 2 "Package_SO:SOIC-8_3.9x4.9mm_P1.27mm" H 3810 7180 50  0001 C CNN
-F 3 "http://www.ti.com/lit/ds/symlink/tlc2272.pdf" H 3810 7180 50  0001 C CNN
-F 4 "TLC2272CD" H 0   0   50  0001 C CNN "manf#"
-	2    3810 7180
-	1    0    0    -1
-$EndComp
 Text Label 3340 7080 2    50   ~ 0
 CO2
@@
 NO2
 Wire Wire Line
-	1780 7100 1930 7100
-Wire Wire Line
 	2530 7200 2560 7200
-Wire Wire Line
-	1930 7300 1880 7300
-Wire Wire Line
-	1880 7300 1880 7450
-Wire Wire Line
-	1880 7450 2560 7450
-Wire Wire Line
-	2560 7450 2560 7200
 Connection ~ 2560 7200
 Wire Wire Line
@@
 	4620 5590 4620 5690
 $Comp
-L citizen_sensor-rescue:ATSAMD21E18A-MU-electroniccats U8
+L citizen_sensor-rescue:ATSAMD21E18A-MU-electroniccats-citizen_sensor-rescue U8
 U 1 1 5C5C9AE3
 P 8000 2300
@@
 	5380 2690 5160 2690
 Connection ~ 5160 2690
+$Comp
+L Amplifier_Operational:OPA1602 U1
+U 1 1 5C6F3F91
+P 2230 7200
+F 0 "U1" H 2300 7460 50  0000 C CNN
+F 1 "TLC2272" H 2390 7360 50  0000 C CNN
+F 2 "Package_SO:SOIC-8_3.9x4.9mm_P1.27mm" H 2230 7200 50  0001 C CNN
+F 3 "http://www.ti.com/lit/ds/symlink/opa1604.pdf" H 2230 7200 50  0001 C CNN
+F 4 "TLC2272CD" H 2230 7200 50  0001 C CNN "manf#"
+	1    2230 7200
+	1    0    0    -1
+$EndComp
+Wire Wire Line
+	1780 7100 1930 7100
+Wire Wire Line
+	1880 7300 1930 7300
+$Comp
+L Amplifier_Operational:OPA1602 U1
+U 2 1 5C700814
+P 3810 7180
+F 0 "U1" H 3810 7547 50  0000 C CNN
+F 1 "TLC2272" H 3810 7456 50  0000 C CNN
+F 2 "Package_SO:SOIC-8_3.9x4.9mm_P1.27mm" H 3810 7180 50  0001 C CNN
+F 3 "http://www.ti.com/lit/ds/symlink/opa1604.pdf" H 3810 7180 50  0001 C CNN
+	2    3810 7180
+	1    0    0    -1
+$EndComp
+$Comp
+L Amplifier_Operational:OPA1602 U1
+U 3 1 5C7008B9
+P 2230 7200
+F 0 "U1" H 2188 7246 50  0000 L CNN
+F 1 "TLC2272" H 2188 7155 50  0000 L CNN
+F 2 "Package_SO:SOIC-8_3.9x4.9mm_P1.27mm" H 2230 7200 50  0001 C CNN
+F 3 "http://www.ti.com/lit/ds/symlink/opa1604.pdf" H 2230 7200 50  0001 C CNN
+	3    2230 7200
+	1    0    0    -1
+$EndComp
+$Comp
+L power:GND #PWR0151
+U 1 1 5C709A87
+P 2130 7500
+F 0 "#PWR0151" H 2130 7250 50  0001 C CNN
+F 1 "GND" H 2135 7327 50  0000 C CNN
+F 2 "" H 2130 7500 50  0001 C CNN
+F 3 "" H 2130 7500 50  0001 C CNN
+	1    2130 7500
+	1    0    0    -1
+$EndComp
+Wire Wire Line
+	1880 7730 2560 7730
+Wire Wire Line
+	2560 7200 2560 7730
+Wire Wire Line
+	1880 7300 1880 7730
+$Comp
+L power:+3.3V #PWR0152
+U 1 1 5C713802
+P 2130 6900
+F 0 "#PWR0152" H 2130 6750 50  0001 C CNN
+F 1 "+3.3V" H 2290 6950 50  0000 C CNN
+F 2 "" H 2130 6900 50  0001 C CNN
+F 3 "" H 2130 6900 50  0001 C CNN
+	1    2130 6900
+	1    0    0    -1
+$EndComp
 $EndSCHEMATC
