File: Hardware/sensorsound.sch (KiCad schematic (older format))
At the start: 20 parts, among them U7 LM324

Commit message: add manf# res cap
Parts:
- C11, C13: manf# (none) -> CC0805KKX5R5BB105
- C12, C14: manf# (none) -> 885012107004
- MK1: footprint Connector_PinHeader_2.54mm:PinHeader_1x02_P2.54mm_Vertical -> TerminalBlock_TE-Connectivity:TerminalBlock_TE_282834-2_1x02_P2.54mm_Horizontal; manf# (none) -> 25R4387
- R10, R18: manf# (none) -> ESR10EZPJ102
- R11, R12, R14, R17: manf# (none) -> ESR10EZPJ103
- R13: manf# (none) -> ERJ-6ENF1003V
- R15: manf# (none) -> CRGP0805F22K
- R16, R19: manf# (none) -> ESR10EZPJ101
- R9: manf# (none) -> RCG08052K20JNEA
- U7: manf# (none) -> LM324DR
Changed lines of the file:
@@
 P 2590 3920
 F 0 "MK1" V 2420 3910 50  0000 L CNN
-F 1 "Microphone" V 2500 3320 50  0000 L CNN
-F 2 "Connector_PinHeader_2.54mm:PinHeader_1x02_P2.54mm_Vertical" V 2590 4020 50  0001 C CNN
-F 3 "~" V 2590 4020 50  0001 C CNN
+F 1 "Microphone" V 2330 3795 50  0000 L CNN
+F 2 "TerminalBlock_TE-Connectivity:TerminalBlock_TE_282834-2_1x02_P2.54mm_Horizontal" V 2590 4020 50  0001 C CNN
+F 3 "http://www.farnell.com/datasheets/1660938.pdf" V 2590 4020 50  0001 C CNN
+F 4 "25R4387" H 0   0   50  0001 C CNN "manf#"
 	1    2590 3920
 	1    0    0    -1
@@
 F 1 "LM324" H 6570 4196 50  0000 C CNN
 F 2 "Package_SO:SOIC-14_3.9x8.7mm_P1.27mm" H 6520 4020 50  0001 C CNN
-F 3 "http://www.ti.com/lit/ds/symlink/lm2902-n.pdf" H 6620 4120 50  0001 C CNN
+F 3 "http://www.ti.com/lit/ds/symlink/lm324.pdf" H 6620 4120 50  0001 C CNN
+F 4 "LM324DR" H 0   0   50  0001 C CNN "manf#"
 	2    6570 3920
 	1    0    0    1
@@
 F 1 "LM324" H 4800 3640 50  0000 C CNN
 F 2 "Package_SO:SOIC-14_3.9x8.7mm_P1.27mm" H 4690 3920 50  0001 C CNN
-F 3 "" H 4790 4020 50  0001 C CNN
+F 3 "http://www.ti.com/lit/ds/symlink/lm324.pdf" H 4790 4020 50  0001 C CNN
+F 4 "LM324DR" H 0   0   50  0001 C CNN "manf#"
 	1    4740 3820
 	1    0    0    1
@@
 F 1 "LM324" H 9050 4096 50  0000 C CNN
 F 2 "Package_SO:SOIC-14_3.9x8.7mm_P1.27mm" H 9000 3920 50  0001 C CNN
-F 3 "http://www.ti.com/lit/ds/symlink/lm2902-n.pdf" H 9100 4020 50  0001 C CNN
+F 3 "http://www.ti.com/lit/ds/symlink/lm324.pdf" H 9100 4020 50  0001 C CNN
+F 4 "LM324DR" H 0   0   50  0001 C CNN "manf#"
 	4    9050 3820
 	1    0    0    1
@@
 F 1 "2.2K" H 2980 3415 50  0000 L CNN
 F 2 "Resistor_SMD:R_0805_2012Metric_Pad1.15x1.40mm_HandSolder" V 2840 3460 50  0001 C CNN
-F 3 "~" H 2910 3460 50  0001 C CNN
+F 3 "https://www.mouser.mx/datasheet/2/427/rcge3-254226.pdf" H 2910 3460 50  0001 C CNN
+F 4 "RCG08052K20JNEA" H 0   0   50  0001 C CNN "manf#"
 	1    2910 3460
 	1    0    0    -1
@@
 F 1 "10uF" V 3150 3720 50  0000 C CNN
 F 2 "Capacitor_SMD:C_0805_2012Metric_Pad1.15x1.40mm_HandSolder" H 3260 3720 50  0001 C CNN
-F 3 "~" H 3260 3720 50  0001 C CNN
+F 3 "https://www.mouser.mx/datasheet/2/445/885012107004-554083.pdf" H 3260 3720 50  0001 C CNN
+F 4 "885012107004" H 0   0   50  0001 C CNN "manf#"
 	1    3260 3720
 	0    -1   -1   0
@@
 F 1 "1K" V 3730 3730 50  0000 C CNN
 F 2 "Resistor_SMD:R_0805_2012Metric_Pad1.15x1.40mm_HandSolder" V 3580 3720 50  0001 C CNN
-F 3 "~" H 3650 3720 50  0001 C CNN
+F 3 "https://www.mouser.mx/datasheet/2/348/esr-e-1139161.pdf" H 3650 3720 50  0001 C CNN
+F 4 "ESR10EZPJ102" H 0   0   50  0001 C CNN "manf#"
 	1    3650 3720
 	0    1    1    0
@@
 F 1 "10K" H 4000 3415 50  0000 L CNN
 F 2 "Resistor_SMD:R_0805_2012Metric_Pad1.15x1.40mm_HandSolder" V 3860 3460 50  0001 C CNN
-F 3 "~" H 3930 3460 50  0001 C CNN
+F 3 "https://www.mouser.mx/datasheet/2/348/esr-e-1139161.pdf" H 3930 3460 50  0001 C CNN
+F 4 "ESR10EZPJ103" H 0   0   50  0001 C CNN "manf#"
 	1    3930 3460
 	1    0    0    -1
@@
 F 1 "10K" H 3860 4205 50  0000 R CNN
 F 2 "Resistor_SMD:R_0805_2012Metric_Pad1.15x1.40mm_HandSolder" V 3860 4160 50  0001 C CNN
-F 3 "~" H 3930 4160 50  0001 C CNN
+F 3 "https://www.mouser.mx/datasheet/2/348/esr-e-1139161.pdf" H 3930 4160 50  0001 C CNN
+F 4 "ESR10EZPJ103" H 0   0   50  0001 C CNN "manf#"
 	1    3930 4160
 	-1   0    0    1
@@
 F 1 "100K" V 4610 3060 50  0000 C CNN
 F 2 "Resistor_SMD:R_0805_2012Metric_Pad1.15x1.40mm_HandSolder" V 4630 3060 50  0001 C CNN
-F 3 "~" H 4700 3060 50  0001 C CNN
+F 3 "https://www.mouser.mx/datasheet/2/315/AOA0000C304-1149620.pdf" H 4700 3060 50  0001 C CNN
+F 4 "ERJ-6ENF1003V" H 0   0   50  0001 C CNN "manf#"
 	1    4700 3060
 	0    -1   -1   0
@@
 F 1 "1uF" V 5220 3820 50  0000 C CNN
 F 2 "Capacitor_SMD:C_0805_2012Metric_Pad1.15x1.40mm_HandSolder" H 5340 3820 50  0001 C CNN
-F 3 "~" H 5340 3820 50  0001 C CNN
+F 3 "https://www.mouser.mx/datasheet/2/447/UPY-GPHC_X5R_4V-to-50V_25-1131599.pdf" H 5340 3820 50  0001 C CNN
+F 4 "CC0805KKX5R5BB105" H 0   0   50  0001 C CNN "manf#"
 	1    5340 3820
 	0    -1   -1   0
@@
 F 1 "LM324" H 4700 3540 50  0000 L CNN
 F 2 "Package_SO:SOIC-14_3.9x8.7mm_P1.27mm" H 4700 3920 50  0001 C CNN
-F 3 "http://www.ti.com/lit/ds/symlink/lm2902-n.pdf" H 4800 4020 50  0001 C CNN
+F 3 "http://www.ti.com/lit/ds/symlink/lm324.pdf" H 4800 4020 50  0001 C CNN
+F 4 "LM324DR" H 0   0   50  0001 C CNN "manf#"
 	5    4750 3820
 	1    0    0    -1
@@
 F 1 "10K" V 5920 3820 50  0000 C CNN
 F 2 "Resistor_SMD:R_0805_2012Metric_Pad1.15x1.40mm_HandSolder" V 5760 3820 50  0001 C CNN
-F 3 "~" H 5830 3820 50  0001 C CNN
+F 3 "https://www.mouser.mx/datasheet/2/348/esr-e-1139161.pdf" H 5830 3820 50  0001 C CNN
+F 4 "ESR10EZPJ103" H 0   0   50  0001 C CNN "manf#"
 	1    5830 3820
 	0    1    1    0
@@
 F 1 "22K" V 6660 3130 50  0000 C CNN
 F 2 "Resistor_SMD:R_0805_2012Metric_Pad1.15x1.40mm_HandSolder" V 6500 3130 50  0001 C CNN
-F 3 "~" H 6570 3130 50  0001 C CNN
+F 3 "https://www.mouser.mx/datasheet/2/418/NG_DS_9-1773463-9_A-1358566.pdf" H 6570 3130 50  0001 C CNN
+F 4 "CRGP0805F22K" H 0   0   50  0001 C CNN "manf#"
 	1    6570 3130
 	0    1    1    0
@@
 F 1 "100" V 7620 3920 50  0000 C CNN
 F 2 "Resistor_SMD:R_0805_2012Metric_Pad1.15x1.40mm_HandSolder" V 7460 3920 50  0001 C CNN
-F 3 "~" H 7530 3920 50  0001 C CNN
+F 3 "https://www.mouser.mx/datasheet/2/348/esr-e-1139161.pdf" H 7530 3920 50  0001 C CNN
+F 4 "ESR10EZPJ101" H 0   0   50  0001 C CNN "manf#"
 	1    7530 3920
 	0    1    1    0
@@
 F 1 "10uF" H 7818 4205 50  0000 R CNN
 F 2 "Capacitor_SMD:C_0805_2012Metric_Pad1.15x1.40mm_HandSolder" H 7910 4160 50  0001 C CNN
-F 3 "~" H 7910 4160 50  0001 C CNN
+F 3 "https://www.mouser.mx/datasheet/2/445/885012107004-554083.pdf" H 7910 4160 50  0001 C CNN
+F 4 "885012107004" H 0   0   50  0001 C CNN "manf#"
 	1    7910 4160
 	-1   0    0    1
@@
 F 1 "10K" H 8310 4190 50  0000 C CNN
 F 2 "Resistor_SMD:R_0805_2012Metric_Pad1.15x1.40mm_HandSolder" V 8360 4160 50  0001 C CNN
-F 3 "~" H 8430 4160 50  0001 C CNN
+F 3 "https://www.mouser.mx/datasheet/2/348/esr-e-1139161.pdf" H 8430 4160 50  0001 C CNN
+F 4 "ESR10EZPJ103" H 0   0   50  0001 C CNN "manf#"
 	1    8430 4160
 	-1   0    0    1
@@
 F 1 "1K" V 8864 3330 50  0000 C CNN
 F 2 "Resistor_SMD:R_0805_2012Metric_Pad1.15x1.40mm_HandSolder" V 8910 3330 50  0001 C CNN
-F 3 "~" H 8980 3330 50  0001 C CNN
+F 3 "https://www.mouser.mx/datasheet/2/348/esr-e-1139161.pdf" H 8980 3330 50  0001 C CNN
+F 4 "ESR10EZPJ102" H 0   0   50  0001 C CNN "manf#"
 	1    8980 3330
 	0    -1   -1   0
@@
 F 1 "100" V 9574 3820 50  0000 C CNN
 F 2 "Resistor_SMD:R_0805_2012Metric_Pad1.15x1.40mm_HandSolder" V 9620 3820 50  0001 C CNN
-F 3 "~" H 9690 3820 50  0001 C CNN
+F 3 "https://www.mouser.mx/datasheet/2/348/esr-e-1139161.pdf" H 9690 3820 50  0001 C CNN
+F 4 "ESR10EZPJ101" H 0   0   50  0001 C CNN "manf#"
 	1    9690 3820
 	0    -1   -1   0
@@
 F 1 "1uf" H 1552 3775 50  0000 L CNN
 F 2 "Capacitor_SMD:C_0805_2012Metric_Pad1.15x1.40mm_HandSolder" H 1460 3820 50  0001 C CNN
-F 3 "~" H 1460 3820 50  0001 C CNN
+F 3 "https://www.mouser.mx/datasheet/2/447/UPY-GPHC_X5R_4V-to-50V_25-1131599.pdf" H 1460 3820 50  0001 C CNN
+F 4 "CC0805KKX5R5BB105" H 0   0   50  0001 C CNN "manf#"
 	1    1460 3820
 	1    0    0    -1
