File: Hardware/_saved_sensorsound.sch (KiCad schematic (older format))
At the start: 21 parts, among them U7 LM324

Commit message: Update schematic
Parts:
- RV1: footprint Potentiometer_THT:Potentiometer_Bourns_3386P_Vertical -> Potentiometer_THT:Potentiometer_Bourns_3386X_Horizontal
Changed lines of the file:
@@
 F 0 "RV1" V 4910 2850 50  0000 C CNN
 F 1 "100K GAIN" V 4620 2770 50  0000 C CNN
-F 2 "Potentiometer_THT:Potentiometer_Bourns_3386P_Vertical" H 4710 2770 50  0001 C CNN
+F 2 "Potentiometer_THT:Potentiometer_Bourns_3386X_Horizontal" H 4710 2770 50  0001 C CNN
 F 3 "https://www.mouser.mx/datasheet/2/54/362-776956.pdf" H 4710 2770 50  0001 C CNN
 F 4 "3362P-1-104LF" H 0   0   50  0001 C CNN "manf#"
