File: Hardware/citizen_sensor.kicad_pcb (KiCad board)
At the start: 2 copper layers, 52 x 80 mm, 76 parts, among them J1 BATT, J2 USB_B_Micro, J3 VEML6075, J4 BME280, J5 PROG, J6 CSS811, J7 MAX30105, Q1 2N7002, SW1 RST, U1 TLC2272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

Commit message: Change On LED
Parts:
- AE1, D3: moved to F.Cu
- moved R8 12.9 mm to (170.8, 60.5), turned to 180 degrees
- moved D3 11.2 mm to (163.7, 59.7)
Routing:
- net VCC: track 63.1 -> 44.9 mm
- net Net-(D3-Pad1): track 2.02 -> 10.0 mm, vias 0 -> 1
- net +3V3: track 347.4 -> 349.4 mm, vias 8 -> 9
- net GND: track 58.8 -> 57.0 mm, vias 16 -> 15
- net Net-(D2-Pad1): track 27.5 -> 26.3 mm
