File: Hardware/citizen_sensor.kicad_pcb (KiCad board)
At the start: 2 copper layers, 52 x 80 mm, 76 parts, among them J1 BATT, J2 USB_B_Micro, J3 VEML6075, J4 BME280, J5 PROG, J6 CSS811, J7 MAX30105, Q1 2N7002, SW1 RST, U1 TLC2272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

Commit message: add led builtin en PCB
Parts:
- added Blink: Builtin, LED_SMD:LED_0805_2012Metric_Castellated, F.Cu at (163.8, 63.5)
- added R24: 330, Resistor_SMD:R_0805_2012Metric_Pad1.15x1.40mm_HandSolder, F.Cu at (163.7, 66.7)
- R6: value 1 -> 47k
- R8: value 1k -> 330
- moved G*** 10.6 mm to (166.2, 75.4)
- moved G*** 2.87 mm to (158.8, 74.8)
Connections:
- net ENVOL renamed /ENVOL
- U8 pad 14: Net-(U8-Pad14) -> /LED_BUILTIN
Routing:
- net /LED_BUILTIN: track 0.00 -> 31.5 mm, vias 0 -> 3
- net Net-(D6-Pad1): track 0.00 -> 3.22 mm
- net /BATTLEVEL: track 74.4 -> 77.1 mm
- net Net-(SW1-Pad2): track 27.0 -> 25.0 mm
- net /DIO0: track 46.1 -> 47.7 mm
- net /DIO2: track 30.5 -> 31.2 mm
- net /ENVOL: track 14.0 -> 14.5 mm

Commit message: Add V0.1 text
Other:
- board text added: "V 0.1"
Changed lines of the file:
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@@
   (general
     (thickness 1.6)
-    (drawings 49)
+    (drawings 50)
     (tracks 743)
     (zones 0)
@@
     )
   )
+  (gr_text "V 0.1" (at 164.13226 69.72554) (layer F.SilkS)
+    (effects (font (size 1.5 1.5) (thickness 0.3)))
+  )
   (gr_arc (start 171 115) (end 171 120) (angle -90) (layer Edge.Cuts) (width 0.15))
   (gr_arc (start 129 115) (end 124 115) (angle -90) (layer Edge.Cuts) (width 0.15))
@@
   (segment (start 151.145 71.335) (end 151.295 71.185) (width 0.3) (layer F.Cu) (net 40))
   (segment (start 148.745 71.335) (end 151.145 71.335) (width 0.3) (layer F.Cu) (net 40))
-  (via (at 151.16 82.39) (size 0.8) (drill 0.4) (layers F.Cu B.Cu) (net 61))
-  (segment (start 151.2 82.43) (end 151.16 82.39) (width 0.5) (layer B.Cu) (net 61))
-  (segment (start 151.2 84.25) (end 151.2 82.43) (width 0.5) (layer B.Cu) (net 61))
   (via (at 134.1 77.9) (size 0.8) (drill 0.4) (layers F.Cu B.Cu) (net 41))
   (segment (start 134.2 78) (end 134.1 77.9) (width 0.3) (layer F.Cu) (net 41))
@@
   (segment (start 155.9433 74.425) (end 160.11398 74.425) (width 0.3) (layer B.Cu) (net 60))
   (segment (start 160.11398 74.425) (end 160.11398 64.35344) (width 0.3) (layer F.Cu) (net 60))
+  (via (at 151.16 82.39) (size 0.8) (drill 0.4) (layers F.Cu B.Cu) (net 61))
+  (segment (start 151.2 82.43) (end 151.16 82.39) (width 0.5) (layer B.Cu) (net 61))
+  (segment (start 151.2 84.25) (end 151.2 82.43) (width 0.5) (layer B.Cu) (net 61))
   (segment (start 151.16 82.39) (end 151.16 73.8586) (width 0.5) (layer F.Cu) (net 61))
   (segment (start 151.16 73.8586) (end 151.87676 73.14184) (width 0.5) (layer F.Cu) (net 61))

Commit message: Update Kicad5 and fix RESET CSS811
Parts:
- renumbered Blink to D6
Connections:
- J6 pad 7: GND -> Net-(J6-Pad7)
Changed lines of the file:
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@@
-(kicad_pcb (version 20171130) (host pcbnew "(5.1.0)-1")
+(kicad_pcb (version 20171130) (host pcbnew "(5.1.5-0-10_14)")
   (general
     (thickness 1.6)
@@
     (zones 0)
     (modules 78)
-    (nets 62)
+    (nets 63)
   )
   (page A4)
@@
   (net 60 /LED_BUILTIN)
   (net 61 /ENVOL)
+  (net 62 "Net-(J6-Pad7)")
   (net_class Default "This is the default net class."
     (clearance 0.25)
@@
     (add_net "Net-(D6-Pad1)")
     (add_net "Net-(F1-Pad1)")
+    (add_net "Net-(J6-Pad7)")
     (add_net "Net-(J6-Pad8)")
     (add_net "Net-(Q1-Pad1)")
@@
       (net 26 /INTCSS))
     (pad 7 thru_hole oval (at 0 15.24 90) (size 1.7 1.7) (drill 1) (layers *.Cu *.Mask)
-      (net 2 GND))
+      (net 62 "Net-(J6-Pad7)"))
     (pad 8 thru_hole oval (at 0 17.78 90) (size 1.7 1.7) (drill 1) (layers *.Cu *.Mask)
       (net 27 "Net-(J6-Pad8)"))
@@
     (tags "LED castellated")
     (attr smd)
-    (fp_text reference Blink (at 4.03622 0.00508 180) (layer F.SilkS)
+    (fp_text reference D6 (at 4.03622 0.00508 180) (layer F.SilkS)
       (effects (font (size 1 1) (thickness 0.15)))
     )

Commit message: update v1.1
Parts:
- removed the G*** at (170.7, 56.7)
- removed the G*** at (169.6, 104.0)
- removed the G*** at (166.2, 75.4)
- removed the G*** at (151.1, 104.5)
- REF***: moved to B.Cu
- moved G*** 20.6 mm to (151.4, 104.1)
- moved G*** 3.23 mm to (162.1, 74.4)
- turned REF*** to 180 degrees
Other:
- board text added: "V1.1"
- board text removed: "V 0.1"

Commit message: update kicad 6
Other:
- net class Default removed
- net class vcc removed
